Commit message: update gazebo

File: urdf/test2.urdf (robot description, URDF)
Before this commit: robot hmr, 7 links, 6 joints
Links:
- added link base, mass 0.0
Joints:
- added joint joint: type fixed, parent base, child base_link, origin xyz=0.0 0.0 1.12 rpy=0.0 0.0 0.0

Commit message: up

File: urdf/test2.urdf (robot description, URDF)
Before this commit: robot hmr, 8 links, 7 joints
Joints:
- joint ljoint1: limit (none) -> lower=-0.6981 upper=1.0472 effort=2.0 velocity=0.2
- joint ljoint2: limit (none) -> lower=-1.0472 upper=0.0 effort=2.0 velocity=0.2
- joint ljoint3: limit (none) -> lower=-0.8727 upper=0.5236 effort=2.0 velocity=0.2
- joint rjoint1: limit (none) -> lower=-0.6981 upper=1.0472 effort=2.0 velocity=0.2
- joint rjoint2: limit (none) -> lower=-1.0472 upper=0.0 effort=2.0 velocity=0.2
- joint rljoint3: limit (none) -> lower=-0.8727 upper=0.5236 effort=2.0 velocity=0.2
