Commit message: update

File: urdf/test2.xacro (robot description, xacro)
@@ -7,5 +7,11 @@
   <!-- <xacro:include filename="$(find hmr)/urdf/materials.xacro" /> -->
   <!-- Import all Gazebo-customization elements, including Gazebo colors -->
-  <xacro:include filename="$(find hmr)/urdf/test2.gazebo" />
+  <!-- <xacro:include filename="$(find hmr)/urdf/test2.gazebo" /> -->
+  <gazebo>
+    <plugin name="gazebo_ros_control" filename="libgazebo_ros_control.so">
+      <robotNamespace>/hmr</robotNamespace>
+      <robotSimType>gazebo_ros_control/DefaultRobotHWSim</robotSimType>
+    </plugin>
+  </gazebo>
   <link name="base">
     <inertial>
@@ -410,3 +416,63 @@
     <limit lower="-0.8727" upper="0.5236" effort="2.0" velocity="0.2"/>
   </joint>
+  <transmission name="ltran1">
+    <type>transmission_interface/SimpleTransmission</type>
+    <joint name="ljoint1">
+      <hardwareInterface>hardware_interface/PositionJointInterface</hardwareInterface>
+    </joint>
+    <actuator name="lmotor1">
+      <mechanicalReduction>1.0</mechanicalReduction>
+      <hardwareInterface>hardware_interface/PositionJointInterface</hardwareInterface>
+    </actuator>
+  </transmission>
+  <transmission name="ltran2">
+    <type>transmission_interface/SimpleTransmission</type>
+    <joint name="ljoint2">
+      <hardwareInterface>hardware_interface/PositionJointInterface</hardwareInterface>
+    </joint>
+    <actuator name="lmotor2">
+      <mechanicalReduction>1.0</mechanicalReduction>
+      <hardwareInterface>hardware_interface/PositionJointInterface</hardwareInterface>
+    </actuator>
+  </transmission>
+  <transmission name="ltran3">
+    <type>transmission_interface/SimpleTransmission</type>
+    <joint name="ljoint3">
+      <hardwareInterface>hardware_interface/PositionJointInterface</hardwareInterface>
+    </joint>
+    <actuator name="lmotor3">
+      <mechanicalReduction>1.0</mechanicalReduction>
+      <hardwareInterface>hardware_interface/PositionJointInterface</hardwareInterface>
+    </actuator>
+  </transmission>
+  <transmission name="rtran1">
+    <type>transmission_interface/SimpleTransmission</type>
+    <joint name="rjoint1">
+      <hardwareInterface>hardware_interface/PositionJointInterface</hardwareInterface>
+    </joint>
+    <actuator name="rmotor1">
+      <mechanicalReduction>1.0</mechanicalReduction>
+      <hardwareInterface>hardware_interface/PositionJointInterface</hardwareInterface>
+    </actuator>
+  </transmission>
+  <transmission name="rtran2">
+    <type>transmission_interface/SimpleTransmission</type>
+    <joint name="rjoint2">
+      <hardwareInterface>hardware_interface/PositionJointInterface</hardwareInterface>
+    </joint>
+    <actuator name="rmotor2">
+      <mechanicalReduction>1.0</mechanicalReduction>
+      <hardwareInterface>hardware_interface/PositionJointInterface</hardwareInterface>
+    </actuator>
+  </transmission>
+  <transmission name="rtran3">
+    <type>transmission_interface/SimpleTransmission</type>
+    <joint name="rjoint3">
+      <hardwareInterface>hardware_interface/PositionJointInterface</hardwareInterface>
+    </joint>
+    <actuator name="rmotor3">
+      <mechanicalReduction>1.0</mechanicalReduction>
+      <hardwareInterface>hardware_interface/PositionJointInterface</hardwareInterface>
+    </actuator>
+  </transmission>
 </robot>

Commit message: update

File: urdf/test2.xacro (robot description, xacro)
@@ -14,4 +14,9 @@
     </plugin>
   </gazebo>
+  <link name="world"/>
+  <joint name="fixed" type="fixed">
+    <parent link="world"/>
+    <child link="base"/>
+  </joint>
   <link name="base">
     <!-- <inertial>

Commit message: update

File: urdf/test2.xacro (robot description, xacro)
@@ -421,12 +421,74 @@
     <limit lower="-0.8727" upper="0.5236" effort="2.0" velocity="0.2"/>
   </joint>
+  <!--  -->
+  <!-- <transmission name="ltran1">
+    <type>transmission_interface/SimpleTransmission</type>
+    <joint name="ljoint1">
+      <hardwareInterface>hardware_interface/EffortJointInterface</hardwareInterface>
+    </joint>
+    <actuator name="lmotor1">
+      <mechanicalReduction>1.0</mechanicalReduction>
+      <hardwareInterface>hardware_interface/EffortJointInterface</hardwareInterface>
+    </actuator>
+  </transmission>
+  <transmission name="ltran2">
+    <type>transmission_interface/SimpleTransmission</type>
+    <joint name="ljoint2">
+      <hardwareInterface>hardware_interface/EffortJointInterface</hardwareInterface>
+    </joint>
+    <actuator name="lmotor2">
+      <mechanicalReduction>1.0</mechanicalReduction>
+      <hardwareInterface>hardware_interface/EffortJointInterface</hardwareInterface>
+    </actuator>
+  </transmission>
+  <transmission name="ltran3">
+    <type>transmission_interface/SimpleTransmission</type>
+    <joint name="ljoint3">
+      <hardwareInterface>hardware_interface/EffortJointInterface</hardwareInterface>
+    </joint>
+    <actuator name="lmotor3">
+      <mechanicalReduction>1.0</mechanicalReduction>
+      <hardwareInterface>hardware_interface/EffortJointInterface</hardwareInterface>
+    </actuator>
+  </transmission>
+  <transmission name="rtran1">
+    <type>transmission_interface/SimpleTransmission</type>
+    <joint name="rjoint1">
+      <hardwareInterface>hardware_interface/EffortJointInterface</hardwareInterface>
+    </joint>
+    <actuator name="rmotor1">
+      <mechanicalReduction>1.0</mechanicalReduction>
+      <hardwareInterface>hardware_interface/EffortJointInterface</hardwareInterface>
+    </actuator>
+  </transmission>
+  <transmission name="rtran2">
+    <type>transmission_interface/SimpleTransmission</type>
+    <joint name="rjoint2">
+      <hardwareInterface>hardware_interface/EffortJointInterface</hardwareInterface>
+    </joint>
+    <actuator name="rmotor2">
+      <mechanicalReduction>1.0</mechanicalReduction>
+      <hardwareInterface>hardware_interface/EffortJointInterface</hardwareInterface>
+    </actuator>
+  </transmission>
+  <transmission name="rtran3">
+    <type>transmission_interface/SimpleTransmission</type>
+    <joint name="rjoint3">
+      <hardwareInterface>hardware_interface/EffortJointInterface</hardwareInterface>
+    </joint>
+    <actuator name="rmotor3">
+      <mechanicalReduction>1.0</mechanicalReduction>
+      <hardwareInterface>hardware_interface/EffortJointInterface</hardwareInterface>
+    </actuator>
+  </transmission> -->
+  <!--  -->
   <transmission name="ltran1">
     <type>transmission_interface/SimpleTransmission</type>
     <joint name="ljoint1">
-      <hardwareInterface>hardware_interface/EffortJointInterface</hardwareInterface>
+      <hardwareInterface>hardware_interface/PositionJointInterface</hardwareInterface>
     </joint>
     <actuator name="lmotor1">
       <mechanicalReduction>1.0</mechanicalReduction>
-      <hardwareInterface>hardware_interface/EffortJointInterface</hardwareInterface>
+      <hardwareInterface>hardware_interface/PositionJointInterface</hardwareInterface>
     </actuator>
   </transmission>
@@ -434,9 +496,9 @@
     <type>transmission_interface/SimpleTransmission</type>
     <joint name="ljoint2">
-      <hardwareInterface>hardware_interface/EffortJointInterface</hardwareInterface>
+      <hardwareInterface>hardware_interface/PositionJointInterface</hardwareInterface>
     </joint>
     <actuator name="lmotor2">
       <mechanicalReduction>1.0</mechanicalReduction>
-      <hardwareInterface>hardware_interface/EffortJointInterface</hardwareInterface>
+      <hardwareInterface>hardware_interface/PositionJointInterface</hardwareInterface>
     </actuator>
   </transmission>
@@ -444,9 +506,9 @@
     <type>transmission_interface/SimpleTransmission</type>
     <joint name="ljoint3">
-      <hardwareInterface>hardware_interface/EffortJointInterface</hardwareInterface>
+      <hardwareInterface>hardware_interface/PositionJointInterface</hardwareInterface>
     </joint>
     <actuator name="lmotor3">
       <mechanicalReduction>1.0</mechanicalReduction>
-      <hardwareInterface>hardware_interface/EffortJointInterface</hardwareInterface>
+      <hardwareInterface>hardware_interface/PositionJointInterface</hardwareInterface>
     </actuator>
   </transmission>
@@ -454,9 +516,9 @@
     <type>transmission_interface/SimpleTransmission</type>
     <joint name="rjoint1">
-      <hardwareInterface>hardware_interface/EffortJointInterface</hardwareInterface>
+      <hardwareInterface>hardware_interface/PositionJointInterface</hardwareInterface>
     </joint>
     <actuator name="rmotor1">
       <mechanicalReduction>1.0</mechanicalReduction>
-      <hardwareInterface>hardware_interface/EffortJointInterface</hardwareInterface>
+      <hardwareInterface>hardware_interface/PositionJointInterface</hardwareInterface>
     </actuator>
   </transmission>
@@ -464,9 +526,9 @@
     <type>transmission_interface/SimpleTransmission</type>
     <joint name="rjoint2">
-      <hardwareInterface>hardware_interface/EffortJointInterface</hardwareInterface>
+      <hardwareInterface>hardware_interface/PositionJointInterface</hardwareInterface>
     </joint>
     <actuator name="rmotor2">
       <mechanicalReduction>1.0</mechanicalReduction>
-      <hardwareInterface>hardware_interface/EffortJointInterface</hardwareInterface>
+      <hardwareInterface>hardware_interface/PositionJointInterface</hardwareInterface>
     </actuator>
   </transmission>
@@ -474,9 +536,9 @@
     <type>transmission_interface/SimpleTransmission</type>
     <joint name="rjoint3">
-      <hardwareInterface>hardware_interface/EffortJointInterface</hardwareInterface>
+      <hardwareInterface>hardware_interface/PositionJointInterface</hardwareInterface>
     </joint>
     <actuator name="rmotor3">
       <mechanicalReduction>1.0</mechanicalReduction>
-      <hardwareInterface>hardware_interface/EffortJointInterface</hardwareInterface>
+      <hardwareInterface>hardware_interface/PositionJointInterface</hardwareInterface>
       <!-- <hardwareInterface>hardware_interface/PositionJointInterface</hardwareInterface>       -->
     </actuator>

Commit message: update

File: urdf/test2.xacro (robot description, xacro)
@@ -83,5 +83,6 @@
     <parent link="base"/>
     <child link="base_link"/>
-    <origin xyz="0.0 0.0 1.12" rpy="0.0 0.0 0.0"/>
+    <origin xyz="0.0 0.0 1.12 " rpy="0.0 0.0 0.0"/>
+    <!-- 1.12 -->
   </joint>
   <!--LLINK1-->
@@ -422,4 +423,65 @@
   </joint>
   <!--  -->
+  <transmission name="ltran1">
+    <type>transmission_interface/SimpleTransmission</type>
+    <joint name="ljoint1">
+      <hardwareInterface>hardware_interface/EffortJointInterface</hardwareInterface>
+    </joint>
+    <actuator name="lmotor1">
+      <mechanicalReduction>1.0</mechanicalReduction>
+      <hardwareInterface>hardware_interface/EffortJointInterface</hardwareInterface>
+    </actuator>
+  </transmission>
+  <transmission name="ltran2">
+    <type>transmission_interface/SimpleTransmission</type>
+    <joint name="ljoint2">
+      <hardwareInterface>hardware_interface/EffortJointInterface</hardwareInterface>
+    </joint>
+    <actuator name="lmotor2">
+      <mechanicalReduction>1.0</mechanicalReduction>
+      <hardwareInterface>hardware_interface/EffortJointInterface</hardwareInterface>
+    </actuator>
+  </transmission>
+  <transmission name="ltran3">
+    <type>transmission_interface/SimpleTransmission</type>
+    <joint name="ljoint3">
+      <hardwareInterface>hardware_interface/EffortJointInterface</hardwareInterface>
+    </joint>
+    <actuator name="lmotor3">
+      <mechanicalReduction>1.0</mechanicalReduction>
+      <hardwareInterface>hardware_interface/EffortJointInterface</hardwareInterface>
+    </actuator>
+  </transmission>
+  <transmission name="rtran1">
+    <type>transmission_interface/SimpleTransmission</type>
+    <joint name="rjoint1">
+      <hardwareInterface>hardware_interface/EffortJointInterface</hardwareInterface>
+    </joint>
+    <actuator name="rmotor1">
+      <mechanicalReduction>1.0</mechanicalReduction>
+      <hardwareInterface>hardware_interface/EffortJointInterface</hardwareInterface>
+    </actuator>
+  </transmission>
+  <transmission name="rtran2">
+    <type>transmission_interface/SimpleTransmission</type>
+    <joint name="rjoint2">
+      <hardwareInterface>hardware_interface/EffortJointInterface</hardwareInterface>
+    </joint>
+    <actuator name="rmotor2">
+      <mechanicalReduction>1.0</mechanicalReduction>
+      <hardwareInterface>hardware_interface/EffortJointInterface</hardwareInterface>
+    </actuator>
+  </transmission>
+  <transmission name="rtran3">
+    <type>transmission_interface/SimpleTransmission</type>
+    <joint name="rjoint3">
+      <hardwareInterface>hardware_interface/EffortJointInterface</hardwareInterface>
+    </joint>
+    <actuator name="rmotor3">
+      <mechanicalReduction>1.0</mechanicalReduction>
+      <hardwareInterface>hardware_interface/EffortJointInterface</hardwareInterface>
+    </actuator>
+  </transmission>
+  <!--  -->
   <!-- <transmission name="ltran1">
     <type>transmission_interface/SimpleTransmission</type>
@@ -429,5 +491,5 @@
     <actuator name="lmotor1">
       <mechanicalReduction>1.0</mechanicalReduction>
-      <hardwareInterface>hardware_interface/EffortJointInterface</hardwareInterface>
+      <hardwareInterface>hardware_interface/PositionJointInterface</hardwareInterface>
     </actuator>
   </transmission>
@@ -439,5 +501,5 @@
     <actuator name="lmotor2">
       <mechanicalReduction>1.0</mechanicalReduction>
-      <hardwareInterface>hardware_interface/EffortJointInterface</hardwareInterface>
+      <hardwareInterface>hardware_interface/PositionJointInterface</hardwareInterface>
     </actuator>
   </transmission>
@@ -449,5 +511,5 @@
     <actuator name="lmotor3">
       <mechanicalReduction>1.0</mechanicalReduction>
-      <hardwareInterface>hardware_interface/EffortJointInterface</hardwareInterface>
+      <hardwareInterface>hardware_interface/PositionJointInterface</hardwareInterface>
     </actuator>
   </transmission>
@@ -459,5 +521,5 @@
     <actuator name="rmotor1">
       <mechanicalReduction>1.0</mechanicalReduction>
-      <hardwareInterface>hardware_interface/EffortJointInterface</hardwareInterface>
+      <hardwareInterface>hardware_interface/PositionJointInterface</hardwareInterface>
     </actuator>
   </transmission>
@@ -469,5 +531,5 @@
     <actuator name="rmotor2">
       <mechanicalReduction>1.0</mechanicalReduction>
-      <hardwareInterface>hardware_interface/EffortJointInterface</hardwareInterface>
+      <hardwareInterface>hardware_interface/PositionJointInterface</hardwareInterface>
     </actuator>
   </transmission>
@@ -479,68 +541,6 @@
     <actuator name="rmotor3">
       <mechanicalReduction>1.0</mechanicalReduction>
-      <hardwareInterface>hardware_interface/EffortJointInterface</hardwareInterface>
+      <hardwareInterface>hardware_interface/PositionJointInterface</hardwareInterface>
     </actuator>
   </transmission> -->
-  <!--  -->
-  <transmission name="ltran1">
-    <type>transmission_interface/SimpleTransmission</type>
-    <joint name="ljoint1">
-      <hardwareInterface>hardware_interface/PositionJointInterface</hardwareInterface>
-    </joint>
-    <actuator name="lmotor1">
-      <mechanicalReduction>1.0</mechanicalReduction>
-      <hardwareInterface>hardware_interface/PositionJointInterface</hardwareInterface>
-    </actuator>
-  </transmission>
-  <transmission name="ltran2">
-    <type>transmission_interface/SimpleTransmission</type>
-    <joint name="ljoint2">
-      <hardwareInterface>hardware_interface/PositionJointInterface</hardwareInterface>
-    </joint>
-    <actuator name="lmotor2">
-      <mechanicalReduction>1.0</mechanicalReduction>
-      <hardwareInterface>hardware_interface/PositionJointInterface</hardwareInterface>
-    </actuator>
-  </transmission>
-  <transmission name="ltran3">
-    <type>transmission_interface/SimpleTransmission</type>
-    <joint name="ljoint3">
-      <hardwareInterface>hardware_interface/PositionJointInterface</hardwareInterface>
-    </joint>
-    <actuator name="lmotor3">
-      <mechanicalReduction>1.0</mechanicalReduction>
-      <hardwareInterface>hardware_interface/PositionJointInterface</hardwareInterface>
-    </actuator>
-  </transmission>
-  <transmission name="rtran1">
-    <type>transmission_interface/SimpleTransmission</type>
-    <joint name="rjoint1">
-      <hardwareInterface>hardware_interface/PositionJointInterface</hardwareInterface>
-    </joint>
-    <actuator name="rmotor1">
-      <mechanicalReduction>1.0</mechanicalReduction>
-      <hardwareInterface>hardware_interface/PositionJointInterface</hardwareInterface>
-    </actuator>
-  </transmission>
-  <transmission name="rtran2">
-    <type>transmission_interface/SimpleTransmission</type>
-    <joint name="rjoint2">
-      <hardwareInterface>hardware_interface/PositionJointInterface</hardwareInterface>
-    </joint>
-    <actuator name="rmotor2">
-      <mechanicalReduction>1.0</mechanicalReduction>
-      <hardwareInterface>hardware_interface/PositionJointInterface</hardwareInterface>
-    </actuator>
-  </transmission>
-  <transmission name="rtran3">
-    <type>transmission_interface/SimpleTransmission</type>
-    <joint name="rjoint3">
-      <hardwareInterface>hardware_interface/PositionJointInterface</hardwareInterface>
-    </joint>
-    <actuator name="rmotor3">
-      <mechanicalReduction>1.0</mechanicalReduction>
-      <hardwareInterface>hardware_interface/PositionJointInterface</hardwareInterface>
-      <!-- <hardwareInterface>hardware_interface/PositionJointInterface</hardwareInterface>       -->
-    </actuator>
-  </transmission>
 </robot>
