Commit message: up

File: hmr_description/urdf/gazebo.urdf (robot description, URDF)
Before this commit: robot hmr, 8 links, 7 joints
Links:
- link base_link: geometry collision mesh filename=package://hmr/hmr_description/meshesbase_link.STL; visual mesh filename=package://hmr/hmr_description/meshesbase_link.STL
- link llink1: geometry collision mesh filename=package://hmr/hmr_description/meshesllink1.STL; visual mesh filename=package://hmr/hmr_description/meshesllink1.STL
- link llink2: geometry collision mesh filename=package://hmr/hmr_description/meshesllink2.STL; visual mesh filename=package://hmr/hmr_description/meshesllink2.STL
- link llink3: geometry collision mesh filename=package://hmr/hmr_description/meshesllink3.STL; visual mesh filename=package://hmr/hmr_description/meshesllink3.STL
- link rlink1: geometry collision mesh filename=package://hmr/hmr_description/meshesrlink1.STL; visual mesh filename=package://hmr/hmr_description/meshesrlink1.STL
- link rlink2: geometry collision mesh filename=package://hmr/hmr_description/meshesrlink2.STL; visual mesh filename=package://hmr/hmr_description/meshesrlink2.STL
- link rlink3: geometry collision mesh filename=package://hmr/hmr_description/meshesrlink3.STL; visual mesh filename=package://hmr/hmr_description/meshesrlink3.STL

File: hmr_description/urdf/test2.xacro (robot description, xacro)
@@ -61,5 +61,5 @@
       <geometry>
         <mesh
-          filename="package://hmr/meshes/base_link.STL" />
+          filename="package://hmr/hmr_description/meshes/base_link.STL" />
       </geometry>
       <material name="red">
@@ -73,5 +73,5 @@
       <geometry>
         <mesh
-          filename="package://hmr/meshes/base_link.STL" />
+          filename="package://hmr/hmr_description/meshes/base_link.STL" />
       </geometry>
     </collision>
@@ -109,5 +109,5 @@
       <geometry>
         <mesh
-          filename="package://hmr/meshes/llink1.STL" />
+          filename="package://hmr/hmr_description/meshes/llink1.STL" />
       </geometry>
       <material name="blue">
@@ -121,5 +121,5 @@
       <geometry>
         <mesh
-          filename="package://hmr/meshes/llink1.STL" />
+          filename="package://hmr/hmr_description/meshes/llink1.STL" />
       </geometry>
     </collision>
@@ -165,5 +165,5 @@
       <geometry>
         <mesh
-          filename="package://hmr/meshes/llink2.STL" />
+          filename="package://hmr/hmr_description/meshes/llink2.STL" />
       </geometry>
       <material name="green">
@@ -177,5 +177,5 @@
       <geometry>
         <mesh
-          filename="package://hmr/meshes/llink2.STL" />
+          filename="package://hmr/hmr_description/meshes/llink2.STL" />
       </geometry>
     </collision>
@@ -221,5 +221,5 @@
       <geometry>
         <mesh
-          filename="package://hmr/meshes/llink3.STL" />
+          filename="package://hmr/hmr_description/meshes/llink3.STL" />
       </geometry>
       <material name="black">
@@ -233,5 +233,5 @@
       <geometry>
         <mesh
-          filename="package://hmr/meshes/llink3.STL" />
+          filename="package://hmr/hmr_description/meshes/llink3.STL" />
       </geometry>
     </collision>
@@ -277,5 +277,5 @@
       <geometry>
         <mesh
-          filename="package://hmr/meshes/rlink1.STL" />
+          filename="package://hmr/hmr_description/meshes/rlink1.STL" />
       </geometry>
       <material name="blue">
@@ -289,5 +289,5 @@
       <geometry>
         <mesh
-          filename="package://hmr/meshes/rlink1.STL" />
+          filename="package://hmr/hmr_description/meshes/rlink1.STL" />
       </geometry>
     </collision>
@@ -333,5 +333,5 @@
       <geometry>
         <mesh
-          filename="package://hmr/meshes/rlink2.STL" />
+          filename="package://hmr/hmr_description/meshes/rlink2.STL" />
       </geometry>
       <material name="green">
@@ -345,5 +345,5 @@
       <geometry>
         <mesh
-          filename="package://hmr/meshes/rlink2.STL" />
+          filename="package://hmr/hmr_description/meshes/rlink2.STL" />
       </geometry>
     </collision>
@@ -389,5 +389,5 @@
       <geometry>
         <mesh
-          filename="package://hmr/meshes/rlink3.STL" />
+          filename="package://hmr/hmr_description/meshes/rlink3.STL" />
       </geometry>
       <material name="black">
@@ -401,5 +401,5 @@
       <geometry>
         <mesh
-          filename="package://hmr/meshes/rlink3.STL" />
+          filename="package://hmr/hmr_description/meshes/rlink3.STL" />
       </geometry>
     </collision>
