Commit message: up

File: hmr_description/urdf/hmr.urdf (robot description, URDF)
Before this commit: robot hmr, 7 links, 6 joints
Links:
- link base_link: geometry collision mesh filename=package://hmr/hmr_description/meshesbase_link.STL; visual mesh filename=package://hmr/hmr_description/meshesbase_link.STL
- link llink1: geometry collision mesh filename=package://hmr/hmr_description/meshesllink1.STL; visual mesh filename=package://hmr/hmr_description/meshesllink1.STL
- link llink2: geometry collision mesh filename=package://hmr/hmr_description/meshesllink2.STL; visual mesh filename=package://hmr/hmr_description/meshesllink2.STL
- link llink3: geometry collision mesh filename=package://hmr/hmr_description/meshesllink3.STL; visual mesh filename=package://hmr/hmr_description/meshesllink3.STL
- link rlink1: geometry collision mesh filename=package://hmr/hmr_description/meshesrlink1.STL; visual mesh filename=package://hmr/hmr_description/meshesrlink1.STL
- link rlink2: geometry collision mesh filename=package://hmr/hmr_description/meshesrlink2.STL; visual mesh filename=package://hmr/hmr_description/meshesrlink2.STL
- link rlink3: geometry collision mesh filename=package://hmr/hmr_description/meshesrlink3.STL; visual mesh filename=package://hmr/hmr_description/meshesrlink3.STL

File: hmr_description/urdf/test.urdf (robot description, URDF)
Before this commit: robot hmr, 8 links, 7 joints
Links:
- link base_link: geometry collision mesh filename=package://hmr/hmr_description/meshesbase_link.STL; visual mesh filename=package://hmr/hmr_description/meshesbase_link.STL
- link llink1: geometry collision mesh filename=package://hmr/hmr_description/meshesllink1.STL; visual mesh filename=package://hmr/hmr_description/meshesllink1.STL
- link llink2: geometry collision mesh filename=package://hmr/hmr_description/meshesllink2.STL; visual mesh filename=package://hmr/hmr_description/meshesllink2.STL
- link llink3: geometry collision mesh filename=package://hmr/hmr_description/meshesllink3.STL; visual mesh filename=package://hmr/hmr_description/meshesllink3.STL
- link rlink1: geometry collision mesh filename=package://hmr/hmr_description/meshesrlink1.STL; visual mesh filename=package://hmr/hmr_description/meshesrlink1.STL
- link rlink2: geometry collision mesh filename=package://hmr/hmr_description/meshesrlink2.STL; visual mesh filename=package://hmr/hmr_description/meshesrlink2.STL
- link rlink3: geometry collision mesh filename=package://hmr/hmr_description/meshesrlink3.STL; visual mesh filename=package://hmr/hmr_description/meshesrlink3.STL

File: hmr_description/urdf/test2.urdf (robot description, URDF)
Before this commit: robot hmr, 8 links, 7 joints
Links:
- link base_link: geometry collision mesh filename=package://hmr/hmr_description/meshesbase_link.STL; visual mesh filename=package://hmr/hmr_description/meshesbase_link.STL
- link llink1: geometry collision mesh filename=package://hmr/hmr_description/meshesllink1.STL; visual mesh filename=package://hmr/hmr_description/meshesllink1.STL
- link llink2: geometry collision mesh filename=package://hmr/hmr_description/meshesllink2.STL; visual mesh filename=package://hmr/hmr_description/meshesllink2.STL
- link llink3: geometry collision mesh filename=package://hmr/hmr_description/meshesllink3.STL; visual mesh filename=package://hmr/hmr_description/meshesllink3.STL
- link rlink1: geometry collision mesh filename=package://hmr/hmr_description/meshesrlink1.STL; visual mesh filename=package://hmr/hmr_description/meshesrlink1.STL
- link rlink2: geometry collision mesh filename=package://hmr/hmr_description/meshesrlink2.STL; visual mesh filename=package://hmr/hmr_description/meshesrlink2.STL
- link rlink3: geometry collision mesh filename=package://hmr/hmr_description/meshesrlink3.STL; visual mesh filename=package://hmr/hmr_description/meshesrlink3.STL
