Commit message: up

File: hmr_description/urdf/test2_not_IMU.xacro (robot description, xacro)
@@ -24,12 +24,53 @@
     <material>Gazebo/Blue</material>
   </gazebo>
+  <!--BASE_LINK-->
+  <link
+    name="base_link">
+    <inertial>
+      <origin
+        xyz="-0.000103296813793522 -0.0184749995894324 -0.00709986514009202"
+        rpy="0 0 0" />
+      <mass
+        value="0.933836944447792" />
+      <inertia
+        ixx="0.00139201398308306"
+        ixy="-2.82901658884336E-12"
+        ixz="4.14929438991966E-12"
+        iyy="0.00736197315629375"
+        iyz="-8.0885885721078E-10"
+        izz="0.00614175111526735" />
+    </inertial>
+    <visual>
+      <origin
+        xyz="0 0 0"
+        rpy="0 0 0" />
+      <geometry>
+        <mesh
+          filename="package://hmr/hmr_description/meshes/base_link.STL" />
+      </geometry>
+      <material name="white">
+        <color rgba="1.0 1.0 1.0 1.0"/>
+      </material>
+    </visual>
+    <collision>
+      <origin
+        xyz="0 0 0"
+        rpy="0 0 0" />
+      <geometry>
+        <mesh
+          filename="package://hmr/hmr_description/meshes/base_link.STL" />
+      </geometry>
+    </collision>
+  </link>
+  <gazebo reference="base_link">
+    <material>Gazebo/Blue</material>
+  </gazebo>
   <joint name="joint" type="fixed">
     <parent link="base"/>
-    <child link="imu_link"/>
+    <child link="base_link"/>
     <origin xyz="0.0 0.0 1.4 " rpy="0.0 0.0 3.1416"/>
     <!-- 1.12 -->
   </joint>
   <!--IMU-->
-  <link name="imu_link"/>
   <gazebo>
     <plugin name="imu_plugin" filename="libgazebo_ros_imu.so">
@@ -42,52 +83,4 @@
     </plugin>
   </gazebo>
-  <!--BASE_LINK-->
-  <link
-    name="base_link">
-    <inertial>
-      <origin
-        xyz="-0.000103296813793522 -0.0184749995894324 -0.00709986514009202"
-        rpy="0 0 0" />
-      <mass
-        value="0.933836944447792" />
-      <inertia
-        ixx="0.00139201398308306"
-        ixy="-2.82901658884336E-12"
-        ixz="4.14929438991966E-12"
-        iyy="0.00736197315629375"
-        iyz="-8.0885885721078E-10"
-        izz="0.00614175111526735" />
-    </inertial>
-    <visual>
-      <origin
-        xyz="0 0 0"
-        rpy="0 0 0" />
-      <geometry>
-        <mesh
-          filename="package://hmr/hmr_description/meshes/base_link.STL" />
-      </geometry>
-      <material name="white">
-        <color rgba="1.0 1.0 1.0 1.0"/>
-      </material>
-    </visual>
-    <collision>
-      <origin
-        xyz="0 0 0"
-        rpy="0 0 0" />
-      <geometry>
-        <mesh
-          filename="package://hmr/hmr_description/meshes/base_link.STL" />
-      </geometry>
-    </collision>
-  </link>
-  <gazebo reference="base_link">
-    <material>Gazebo/Blue</material>
-  </gazebo>
-  <joint name="joint" type="fixed">
-    <parent link="imu_link"/>
-    <child link="base_link"/>
-    <origin xyz="0.0 0.0 1.4 " rpy="0.0 0.0 3.1416"/>
-    <!-- 1.12 -->
-  </joint>
   <!--LLINK1-->
   <link

Commit message: up

File: hmr_description/urdf/test2_not_IMU.xacro (robot description, xacro)
@@ -24,4 +24,10 @@
     <material>Gazebo/Blue</material>
   </gazebo>
+  <joint name="imu_joint" type="fixed">
+    <parent link="base"/>
+    <child link="base_link"/>
+    <origin xyz="0.0 0.0 1.4 " rpy="0.0 0.0 3.1416"/>
+    <!-- 1.12 -->
+  </joint>
   <!--BASE_LINK-->
   <link
@@ -29,15 +35,15 @@
     <inertial>
       <origin
-        xyz="-0.000103296813793522 -0.0184749995894324 -0.00709986514009202"
-        rpy="0 0 0" />
-      <mass
-        value="0.933836944447792" />
-      <inertia
-        ixx="0.00139201398308306"
-        ixy="-2.82901658884336E-12"
-        ixz="4.14929438991966E-12"
-        iyy="0.00736197315629375"
-        iyz="-8.0885885721078E-10"
-        izz="0.00614175111526735" />
+        xyz="-8.1485E-05 0.040306 -0.00093209"
+        rpy="0 0 0" />
+      <mass
+        value="2.4018" />
+      <inertia
+        ixx="0.0070769"
+        ixy="-2.7325E-07"
+        ixz="1.9337E-07"
+        iyy="0.015485"
+        iyz="-1.2071E-07"
+        izz="0.009591" />
     </inertial>
     <visual>
@@ -72,15 +78,4 @@
     <!-- 1.12 -->
   </joint>
-  <!--IMU-->
-  <gazebo>
-    <plugin name="imu_plugin" filename="libgazebo_ros_imu.so">
-      <alwaysOn>true</alwaysOn>
-      <bodyName>base</bodyName>
-      <topicName>imu</topicName>
-      <serviceName>imu_service</serviceName>
-      <gaussianNoise>0.0</gaussianNoise>
-      <updateRate>20.0</updateRate>
-    </plugin>
-  </gazebo>
   <!--LLINK1-->
   <link
@@ -88,15 +83,15 @@
     <inertial>
       <origin
-        xyz="0.0499999851262689 -0.248500614775013 5.33671345059814E-05"
-        rpy="0 0 0" />
-      <mass
-        value="0.509664464543895" />
-      <inertia
-        ixx="0.00405279295169879"
-        ixy="-5.17821013423379E-16"
-        ixz="-1.86028405386162E-17"
-        iyy="0.000257140430774596"
-        iyz="2.20410095949559E-06"
-        izz="0.0041884713527824" />
+        xyz="0.056084 -0.21548 -1.1057E-06"
+        rpy="0 0 0" />
+      <mass
+        value="0.43137" />
+      <inertia
+        ixx="0.0026126"
+        ixy="-1.5474E-07"
+        ixz="-5.4626E-08"
+        iyy="0.00020436"
+        iyz="-9.8E-06"
+        izz="0.0027266" />
     </inertial>
     <visual>
@@ -129,5 +124,5 @@
     type="revolute">
     <origin
-      xyz="0.12 0.06 -0.06"
+      xyz="0.1135 0.04 -0.06"
       rpy="1.5708 0 0" />
     <parent
@@ -145,15 +140,15 @@
     <inertial>
       <origin
-        xyz="0.0500545282509017 -0.234393633663144 0.00550026352716933"
-        rpy="0 0 0" />
-      <mass
-        value="0.442265777754145" />
-      <inertia
-        ixx="0.0040117979862963"
-        ixy="-5.09697896497051E-16"
-        ixz="-2.77164071387431E-17"
-        iyy="0.000241596436981563"
-        iyz="-1.10278899850188E-06"
-        izz="0.00416183117175302" />
+        xyz="0.054446 -0.17796 -0.0015786"
+        rpy="0 0 0" />
+      <mass
+        value="0.45541" />
+      <inertia
+        ixx="0.002625"
+        ixy="6.5245E-19"
+        ixz="-3.637E-17"
+        iyy="0.00023283"
+        iyz="4.9149E-06"
+        izz="0.0027437" />
     </inertial>
     <visual>
@@ -186,5 +181,5 @@
     type="revolute">
     <origin
-      xyz="0 -0.5 0"
+      xyz="0 -0.438 0"
       rpy="0 0 0" />
     <parent
@@ -202,15 +197,15 @@
     <inertial>
       <origin
-        xyz="0.0501466994062446 -0.0351041894822217 0.0405185729509365"
-        rpy="0 0 0" />
-      <mass
-        value="0.164387087553345" />
-      <inertia
-        ixx="0.000390399624612182"
-        ixy="6.46553823154572E-18"
-        ixz="7.16521493881578E-17"
-        iyy="0.000442516689346383"
-        iyz="-8.18654011913839E-11"
-        izz="8.27552994226968E-05" />
+        xyz="0.049198 -0.036675 0.049331"
+        rpy="0 0 0" />
+      <mass
+        value="0.29119" />
+      <inertia
+        ixx="0.00061049"
+        ixy="1.3662E-07"
+        ixz="-9.6685E-08"
+        iyy="0.00068435"
+        iyz="-6.0356E-08"
+        izz="0.00011606" />
     </inertial>
     <visual>
@@ -243,5 +238,5 @@
     type="revolute">
     <origin
-      xyz="0 -0.5 0"
+      xyz="0.00735 -0.44 0"
       rpy="0 0 0" />
     <parent
@@ -259,15 +254,15 @@
     <inertial>
       <origin
-        xyz="-0.0500000148736693 -0.248500614774999 5.33671345059189E-05"
-        rpy="0 0 0" />
-      <mass
-        value="0.509664464543895" />
-      <inertia
-        ixx="0.00405279295169879"
-        ixy="-5.17781100332924E-16"
-        ixz="-1.86069004433025E-17"
-        iyy="0.000257140430774596"
-        iyz="2.20410095949557E-06"
-        izz="0.0041884713527824" />
+        xyz="-0.046266 -0.21548 -1.1057E-06"
+        rpy="0 0 0" />
+      <mass
+        value="0.43137" />
+      <inertia
+        ixx="0.0026126"
+        ixy="-1.5474E-07"
+        ixz="-5.4626E-08"
+        iyy="0.00020436"
+        iyz="-9.8E-06"
+        izz="0.0027266" />
     </inertial>
     <visual>
@@ -300,5 +295,5 @@
     type="revolute">
     <origin
-      xyz="-0.12 0.06 -0.06"
+      xyz="-0.12415 0.04 -0.06"
       rpy="1.5708 0 0" />
     <parent
@@ -316,15 +311,15 @@
     <inertial>
       <origin
-        xyz="-0.049945471749016 -0.234393633663131 0.00550026352714499"
-        rpy="0 0 0" />
-      <mass
-        value="0.442265777754145" />
-      <inertia
-        ixx="0.00401179798629629"
-        ixy="-5.09803878440693E-16"
-        ixz="-2.77168469663556E-17"
-        iyy="0.000241596436981563"
-        iyz="-1.10278899850179E-06"
-        izz="0.00416183117175302" />
+        xyz="-0.047904 -0.17796 -0.0015786"
+        rpy="0 0 0" />
+      <mass
+        value="0.45541" />
+      <inertia
+        ixx="0.002625"
+        ixy="6.3076E-19"
+        ixz="-3.6373E-17"
+        iyy="0.00023283"
+        iyz="4.9149E-06"
+        izz="0.0027437" />
     </inertial>
     <visual>
@@ -357,5 +352,5 @@
     type="revolute">
     <origin
-      xyz="0 -0.5 0"
+      xyz="0 -0.438 0"
       rpy="0 0 0" />
     <parent
@@ -373,15 +368,15 @@
     <inertial>
       <origin
-        xyz="-0.0498532993324217 -0.0351041894822506 0.040518572950845"
-        rpy="0 0 0" />
-      <mass
-        value="0.164387087553345" />
-      <inertia
-        ixx="0.000390399624612182"
-        ixy="6.46331811347987E-18"
-        ixz="7.16490435411506E-17"
-        iyy="0.000442516689346383"
-        iyz="-8.18654011935542E-11"
-        izz="8.27552994226968E-05" />
+        xyz="-0.045802 -0.036675 0.049331"
+        rpy="0 0 0" />
+      <mass
+        value="0.29119" />
+      <inertia
+        ixx="0.00061049"
+        ixy="1.3662E-07"
+        ixz="-9.6685E-08"
+        iyy="0.00068435"
+        iyz="-6.0356E-08"
+        izz="0.00011606" />
     </inertial>
     <visual>
@@ -414,5 +409,5 @@
     type="revolute">
     <origin
-      xyz="0 -0.5 0"
+      xyz="0 -0.44 0"
       rpy="0 0 0" />
     <parent
