Commit message: update limit revolute

File: hmr_description/urdf/test2.xacro (robot description, xacro)
@@ -63,6 +63,6 @@
           filename="package://hmr/hmr_description/meshes/base_link.STL" />
       </geometry>
-      <material name="red">
-        <color rgba="1.0 0.0 0.0 1.0"/>
+      <material name="white">
+        <color rgba="1.0 1.0 1.0 1.0"/>
       </material>
     </visual>
@@ -130,5 +130,5 @@
   <joint
     name="ljoint1"
-    type="continuous">
+    type="revolute">
     <origin
       xyz="0.12 0.06 -0.06"
@@ -140,5 +140,5 @@
     <axis
       xyz="1 0 0" />
-    <limit lower="-0.6981" upper="1.0472" effort="2.0" velocity="0.2"/>
+    <limit lower="-0.6981" upper="0.5236" effort="2.0" velocity="0.2"/>
   </joint>
   <!--LLINK2-->
@@ -186,5 +186,5 @@
   <joint
     name="ljoint2"
-    type="continuous">
+    type="revolute">
     <origin
       xyz="0 -0.5 0"
@@ -196,5 +196,5 @@
     <axis
       xyz="1 0 0" />
-    <limit lower="-1.0472" upper="0.0" effort="2.0" velocity="0.2"/>
+    <limit lower="0.0" upper="1.0472" effort="2.0" velocity="0.2"/>
   </joint>
   <!--LLINK3-->
@@ -223,6 +223,6 @@
           filename="package://hmr/hmr_description/meshes/llink3.STL" />
       </geometry>
-      <material name="black">
-        <color rgba="0.0 0.0 0.0 1.0"/>
+      <material name="red">
+        <color rgba="1.0 0.0 0.0 1.0"/>
       </material>
     </visual>
@@ -242,5 +242,5 @@
   <joint
     name="ljoint3"
-    type="continuous">
+    type="revolute">
     <origin
       xyz="0 -0.5 0"
@@ -252,5 +252,5 @@
     <axis
       xyz="1 0 0" />
-    <limit lower="-0.8727" upper="0.5236" effort="2.0" velocity="0.2"/>
+    <limit lower="-0.5236" upper="0.8727" effort="2.0" velocity="0.2"/>
   </joint>
   <!--RLINK1-->
@@ -298,5 +298,5 @@
   <joint
     name="rjoint1"
-    type="continuous">
+    type="revolute">
     <origin
       xyz="-0.12 0.06 -0.06"
@@ -308,5 +308,5 @@
     <axis
       xyz="1 0 0" />
-    <limit lower="-0.6981" upper="1.0472" effort="2.0" velocity="0.2"/>
+    <limit lower="-0.6981" upper="0.5236" effort="2.0" velocity="0.2"/>
   </joint>
   <!--RLINK2-->
@@ -354,5 +354,5 @@
   <joint
     name="rjoint2"
-    type="continuous">
+    type="revolute">
     <origin
       xyz="0 -0.5 0"
@@ -364,5 +364,5 @@
     <axis
       xyz="1 0 0" />
-    <limit lower="-1.0472" upper="0.0" effort="2.0" velocity="0.2"/>
+    <limit lower="0.0" upper="1.0472" effort="2.0" velocity="0.2"/>
   </joint>
   <!--RLINK3-->
@@ -391,6 +391,6 @@
           filename="package://hmr/hmr_description/meshes/rlink3.STL" />
       </geometry>
-      <material name="black">
-        <color rgba="0.0 0.0 0.0 1.0"/>
+      <material name="red">
+        <color rgba="1.0 0.0 0.0 1.0"/>
       </material>
     </visual>
@@ -410,5 +410,5 @@
   <joint
     name="rjoint3"
-    type="continuous">
+    type="revolute">
     <origin
       xyz="0 -0.5 0"
@@ -420,5 +420,5 @@
     <axis
       xyz="1 0 0" />
-    <limit lower="-0.8727" upper="0.5236" effort="2.0" velocity="0.2"/>
+    <limit lower="-0.5236" upper="0.8727" effort="2.0" velocity="0.2"/>
   </joint>
   <!--  -->

Commit message: up

File: hmr_description/urdf/test2.xacro (robot description, xacro)
@@ -69,5 +69,5 @@
     <parent link="base"/>
     <child link="base_link"/>
-    <origin xyz="0.0 0.0 1.12 " rpy="0.0 0.0 0.0"/>
+    <origin xyz="0.0 0.0 1.12 " rpy="0.0 0.0 3.1416"/>
     <!-- 1.12 -->
   </joint>

Commit message: update

File: hmr_description/urdf/test2.xacro (robot description, xacro)
@@ -69,5 +69,5 @@
     <parent link="base"/>
     <child link="base_link"/>
-    <origin xyz="0.0 0.0 1.2 " rpy="0.0 0.0 3.1416"/>
+    <origin xyz="0.0 0.0 1.4 " rpy="0.0 0.0 3.1416"/>
     <!-- 1.12 -->
   </joint>

Commit message: up

File: hmr_description/urdf/test2.xacro (robot description, xacro)
@@ -469,64 +469,3 @@
     </actuator>
   </transmission>
-  <!--  -->
-  <!-- <transmission name="ltran1">
-    <type>transmission_interface/SimpleTransmission</type>
-    <joint name="ljoint1">
-      <hardwareInterface>hardware_interface/EffortJointInterface</hardwareInterface>
-    </joint>
-    <actuator name="lmotor1">
-      <mechanicalReduction>1.0</mechanicalReduction>
-      <hardwareInterface>hardware_interface/PositionJointInterface</hardwareInterface>
-    </actuator>
-  </transmission>
-  <transmission name="ltran2">
-    <type>transmission_interface/SimpleTransmission</type>
-    <joint name="ljoint2">
-      <hardwareInterface>hardware_interface/EffortJointInterface</hardwareInterface>
-    </joint>
-    <actuator name="lmotor2">
-      <mechanicalReduction>1.0</mechanicalReduction>
-      <hardwareInterface>hardware_interface/PositionJointInterface</hardwareInterface>
-    </actuator>
-  </transmission>
-  <transmission name="ltran3">
-    <type>transmission_interface/SimpleTransmission</type>
-    <joint name="ljoint3">
-      <hardwareInterface>hardware_interface/EffortJointInterface</hardwareInterface>
-    </joint>
-    <actuator name="lmotor3">
-      <mechanicalReduction>1.0</mechanicalReduction>
-      <hardwareInterface>hardware_interface/PositionJointInterface</hardwareInterface>
-    </actuator>
-  </transmission>
-  <transmission name="rtran1">
-    <type>transmission_interface/SimpleTransmission</type>
-    <joint name="rjoint1">
-      <hardwareInterface>hardware_interface/EffortJointInterface</hardwareInterface>
-    </joint>
-    <actuator name="rmotor1">
-      <mechanicalReduction>1.0</mechanicalReduction>
-      <hardwareInterface>hardware_interface/PositionJointInterface</hardwareInterface>
-    </actuator>
-  </transmission>
-  <transmission name="rtran2">
-    <type>transmission_interface/SimpleTransmission</type>
-    <joint name="rjoint2">
-      <hardwareInterface>hardware_interface/EffortJointInterface</hardwareInterface>
-    </joint>
-    <actuator name="rmotor2">
-      <mechanicalReduction>1.0</mechanicalReduction>
-      <hardwareInterface>hardware_interface/PositionJointInterface</hardwareInterface>
-    </actuator>
-  </transmission>
-  <transmission name="rtran3">
-    <type>transmission_interface/SimpleTransmission</type>
-    <joint name="rjoint3">
-      <hardwareInterface>hardware_interface/EffortJointInterface</hardwareInterface>
-    </joint>
-    <actuator name="rmotor3">
-      <mechanicalReduction>1.0</mechanicalReduction>
-      <hardwareInterface>hardware_interface/PositionJointInterface</hardwareInterface>
-    </actuator>
-  </transmission> -->
 </robot>

Commit message: update

File: hmr_description/urdf/test2.xacro (robot description, xacro)
@@ -24,4 +24,15 @@
     <material>Gazebo/Blue</material>
   </gazebo>
+  <!--IMU-->
+  <gazebo>
+    <plugin name="imu_plugin" filename="libgazebo_ros_imu.so">
+      <alwaysOn>true</alwaysOn>
+      <bodyName>base</bodyName>
+      <topicName>imu</topicName>
+      <serviceName>imu_service</serviceName>
+      <gaussianNoise>0.0</gaussianNoise>
+      <updateRate>20.0</updateRate>
+    </plugin>
+  </gazebo>
   <!--BASE_LINK-->
   <link
@@ -127,4 +138,5 @@
       xyz="1 0 0" />
     <limit lower="-0.6981" upper="0.5236" effort="2.0" velocity="0.2"/>
+    <!-- <safety_controller soft_lower_limit="" soft_upper_limit="" k_position="" k_velocity=""/> -->
   </joint>
   <!--LLINK2-->
@@ -183,4 +195,5 @@
       xyz="1 0 0" />
     <limit lower="0.0" upper="1.0472" effort="2.0" velocity="0.2"/>
+    <!-- <safety_controller soft_lower_limit="" soft_upper_limit="" k_position="" k_velocity=""/> -->
   </joint>
   <!--LLINK3-->
@@ -238,5 +251,6 @@
     <axis
       xyz="1 0 0" />
-    <limit lower="-0.5236" upper="0.8727" effort="2.0" velocity="0.2"/>
+    <limit lower="-0.3491" upper="0.8727" effort="2.0" velocity="0.2"/>
+    <!-- <safety_controller soft_lower_limit="" soft_upper_limit="" k_position="" k_velocity=""/> -->
   </joint>
   <!--RLINK1-->
@@ -295,4 +309,5 @@
       xyz="1 0 0" />
     <limit lower="-0.6981" upper="0.5236" effort="2.0" velocity="0.2"/>
+    <!-- <safety_controller soft_lower_limit="" soft_upper_limit="" k_position="" k_velocity=""/> -->
   </joint>
   <!--RLINK2-->
@@ -351,4 +366,5 @@
       xyz="1 0 0" />
     <limit lower="0.0" upper="1.0472" effort="2.0" velocity="0.2"/>
+    <!-- <safety_controller soft_lower_limit="" soft_upper_limit="" k_position="" k_velocity=""/> -->
   </joint>
   <!--RLINK3-->
@@ -406,5 +422,6 @@
     <axis
       xyz="1 0 0" />
-    <limit lower="-0.5236" upper="0.8727" effort="2.0" velocity="0.2"/>
+    <limit lower="-0.3491" upper="0.8727" effort="2.0" velocity="0.2"/>
+    <!-- <safety_controller soft_lower_limit="" soft_upper_limit="" k_position="" k_velocity=""/> -->
   </joint>
   <!--  -->

Commit message: up

File: hmr_description/urdf/test2.xacro (robot description, xacro)
@@ -24,5 +24,5 @@
     <material>Gazebo/Blue</material>
   </gazebo>
-  <joint name="joint" type="fixed">
+  <joint name="imu_joint" type="fixed">
     <parent link="base"/>
     <child link="imu_link"/>
@@ -32,8 +32,14 @@
   <!--IMU-->
   <link name="imu_link"/>
+  <gazebo reference="imu_link">
+    <sensor type="imu" name="imu">
+      <always_on>true</always_on>
+    </sensor>
+    <material>Gazebo/FlatBlack</material>
+  </gazebo>
   <gazebo>
     <plugin name="imu_plugin" filename="libgazebo_ros_imu.so">
       <alwaysOn>true</alwaysOn>
-      <bodyName>base</bodyName>
+      <bodyName>imu_link</bodyName>
       <topicName>imu</topicName>
       <serviceName>imu_service</serviceName>
@@ -85,5 +91,5 @@
   </gazebo>
   <joint name="joint" type="fixed">
-    <parent link="imu_link"/>
+    <parent link="base"/>
     <child link="base_link"/>
     <origin xyz="0.0 0.0 1.4 " rpy="0.0 0.0 3.1416"/>
