Commit message: update

File: hmr_description/urdf/test2.xacro (robot description, xacro)
@@ -53,15 +53,15 @@
     <inertial>
       <origin
-        xyz="-0.000103296813793522 -0.0184749995894324 -0.00709986514009202"
-        rpy="0 0 0" />
-      <mass
-        value="0.933836944447792" />
-      <inertia
-        ixx="0.00139201398308306"
-        ixy="-2.82901658884336E-12"
-        ixz="4.14929438991966E-12"
-        iyy="0.00736197315629375"
-        iyz="-8.0885885721078E-10"
-        izz="0.00614175111526735" />
+        xyz="-8.1485E-05 0.040306 -0.00093209"
+        rpy="0 0 0" />
+      <mass
+        value="2.4018" />
+      <inertia
+        ixx="0.0070769"
+        ixy="-2.7325E-07"
+        ixz="1.9337E-07"
+        iyy="0.015485"
+        iyz="-1.2071E-07"
+        izz="0.009591" />
     </inertial>
     <visual>
@@ -101,15 +101,15 @@
     <inertial>
       <origin
-        xyz="0.0499999851262689 -0.248500614775013 5.33671345059814E-05"
-        rpy="0 0 0" />
-      <mass
-        value="0.509664464543895" />
-      <inertia
-        ixx="0.00405279295169879"
-        ixy="-5.17821013423379E-16"
-        ixz="-1.86028405386162E-17"
-        iyy="0.000257140430774596"
-        iyz="2.20410095949559E-06"
-        izz="0.0041884713527824" />
+        xyz="0.056084 -0.21548 -1.1057E-06"
+        rpy="0 0 0" />
+      <mass
+        value="0.43137" />
+      <inertia
+        ixx="0.0026126"
+        ixy="-1.5474E-07"
+        ixz="-5.4626E-08"
+        iyy="0.00020436"
+        iyz="-9.8E-06"
+        izz="0.0027266" />
     </inertial>
     <visual>
@@ -142,5 +142,5 @@
     type="revolute">
     <origin
-      xyz="0.12 0.06 -0.06"
+      xyz="0.1135 0.04 -0.06"
       rpy="1.5708 0 0" />
     <parent
@@ -158,15 +158,15 @@
     <inertial>
       <origin
-        xyz="0.0500545282509017 -0.234393633663144 0.00550026352716933"
-        rpy="0 0 0" />
-      <mass
-        value="0.442265777754145" />
-      <inertia
-        ixx="0.0040117979862963"
-        ixy="-5.09697896497051E-16"
-        ixz="-2.77164071387431E-17"
-        iyy="0.000241596436981563"
-        iyz="-1.10278899850188E-06"
-        izz="0.00416183117175302" />
+        xyz="0.054446 -0.17796 -0.0015786"
+        rpy="0 0 0" />
+      <mass
+        value="0.45541" />
+      <inertia
+        ixx="0.002625"
+        ixy="6.5245E-19"
+        ixz="-3.637E-17"
+        iyy="0.00023283"
+        iyz="4.9149E-06"
+        izz="0.0027437" />
     </inertial>
     <visual>
@@ -199,5 +199,5 @@
     type="revolute">
     <origin
-      xyz="0 -0.5 0"
+      xyz="0 -0.438 0"
       rpy="0 0 0" />
     <parent
@@ -215,15 +215,15 @@
     <inertial>
       <origin
-        xyz="0.0501466994062446 -0.0351041894822217 0.0405185729509365"
-        rpy="0 0 0" />
-      <mass
-        value="0.164387087553345" />
-      <inertia
-        ixx="0.000390399624612182"
-        ixy="6.46553823154572E-18"
-        ixz="7.16521493881578E-17"
-        iyy="0.000442516689346383"
-        iyz="-8.18654011913839E-11"
-        izz="8.27552994226968E-05" />
+        xyz="0.049198 -0.036675 0.049331"
+        rpy="0 0 0" />
+      <mass
+        value="0.29119" />
+      <inertia
+        ixx="0.00061049"
+        ixy="1.3662E-07"
+        ixz="-9.6685E-08"
+        iyy="0.00068435"
+        iyz="-6.0356E-08"
+        izz="0.00011606" />
     </inertial>
     <visual>
@@ -256,5 +256,5 @@
     type="revolute">
     <origin
-      xyz="0 -0.5 0"
+      xyz="0.00735 -0.44 0"
       rpy="0 0 0" />
     <parent
@@ -272,15 +272,15 @@
     <inertial>
       <origin
-        xyz="-0.0500000148736693 -0.248500614774999 5.33671345059189E-05"
-        rpy="0 0 0" />
-      <mass
-        value="0.509664464543895" />
-      <inertia
-        ixx="0.00405279295169879"
-        ixy="-5.17781100332924E-16"
-        ixz="-1.86069004433025E-17"
-        iyy="0.000257140430774596"
-        iyz="2.20410095949557E-06"
-        izz="0.0041884713527824" />
+        xyz="-0.046266 -0.21548 -1.1057E-06"
+        rpy="0 0 0" />
+      <mass
+        value="0.43137" />
+      <inertia
+        ixx="0.0026126"
+        ixy="-1.5474E-07"
+        ixz="-5.4626E-08"
+        iyy="0.00020436"
+        iyz="-9.8E-06"
+        izz="0.0027266" />
     </inertial>
     <visual>
@@ -313,5 +313,5 @@
     type="revolute">
     <origin
-      xyz="-0.12 0.06 -0.06"
+      xyz="-0.12415 0.04 -0.06"
       rpy="1.5708 0 0" />
     <parent
@@ -329,15 +329,15 @@
     <inertial>
       <origin
-        xyz="-0.049945471749016 -0.234393633663131 0.00550026352714499"
-        rpy="0 0 0" />
-      <mass
-        value="0.442265777754145" />
-      <inertia
-        ixx="0.00401179798629629"
-        ixy="-5.09803878440693E-16"
-        ixz="-2.77168469663556E-17"
-        iyy="0.000241596436981563"
-        iyz="-1.10278899850179E-06"
-        izz="0.00416183117175302" />
+        xyz="-0.047904 -0.17796 -0.0015786"
+        rpy="0 0 0" />
+      <mass
+        value="0.45541" />
+      <inertia
+        ixx="0.002625"
+        ixy="6.3076E-19"
+        ixz="-3.6373E-17"
+        iyy="0.00023283"
+        iyz="4.9149E-06"
+        izz="0.0027437" />
     </inertial>
     <visual>
@@ -370,5 +370,5 @@
     type="revolute">
     <origin
-      xyz="0 -0.5 0"
+      xyz="0 -0.438 0"
       rpy="0 0 0" />
     <parent
@@ -386,15 +386,15 @@
     <inertial>
       <origin
-        xyz="-0.0498532993324217 -0.0351041894822506 0.040518572950845"
-        rpy="0 0 0" />
-      <mass
-        value="0.164387087553345" />
-      <inertia
-        ixx="0.000390399624612182"
-        ixy="6.46331811347987E-18"
-        ixz="7.16490435411506E-17"
-        iyy="0.000442516689346383"
-        iyz="-8.18654011935542E-11"
-        izz="8.27552994226968E-05" />
+        xyz="-0.045802 -0.036675 0.049331"
+        rpy="0 0 0" />
+      <mass
+        value="0.29119" />
+      <inertia
+        ixx="0.00061049"
+        ixy="1.3662E-07"
+        ixz="-9.6685E-08"
+        iyy="0.00068435"
+        iyz="-6.0356E-08"
+        izz="0.00011606" />
     </inertial>
     <visual>
@@ -427,5 +427,5 @@
     type="revolute">
     <origin
-      xyz="0 -0.5 0"
+      xyz="0 -0.44 0"
       rpy="0 0 0" />
     <parent

File: hmr_description/urdf/test2_ver2.xacro (robot description, xacro)
@@ -11,26 +11,41 @@
     <plugin name="gazebo_ros_control" filename="libgazebo_ros_control.so">
       <robotNamespace>/hmr</robotNamespace>
-      <robotSimType>gazebo_ros_control/DefaultRobotHWSim</robotSimType>
+      <!-- <robotSimType>gazebo_ros_control/DefaultRobotHWSim</robotSimType> -->
     </plugin>
   </gazebo>
+  <link name="world"/>
+  <joint name="fixed" type="fixed">
+    <parent link="world"/>
+    <child link="base"/>
+  </joint>
   <link name="base">
-    <!-- <inertial>
-      <origin
-        xyz="0.0 0.0 0.0"
-        rpy="0 0 0" />
-      <mass
-        value="0.0" />
-      <inertia
-        ixx="0.0"
-        ixy="0.0"
-        ixz="0.0"
-        iyy="0.0"
-        iyz="0.0"
-        izz="0.0" />
-    </inertial>     -->
   </link>
   <gazebo reference="base">
     <material>Gazebo/Blue</material>
   </gazebo>
+  <joint name="imu_joint" type="fixed">
+    <parent link="base"/>
+    <child link="imu_link"/>
+    <origin xyz="0.0 0.0 1.4 " rpy="0.0 0.0 3.1416"/>
+    <!-- 1.12 -->
+  </joint>
+  <!--IMU-->
+  <link name="imu_link"/>
+  <gazebo reference="imu_link">
+    <sensor type="imu" name="imu">
+      <always_on>true</always_on>
+    </sensor>
+    <material>Gazebo/FlatBlack</material>
+  </gazebo>
+  <gazebo>
+    <plugin name="imu_plugin" filename="libgazebo_ros_imu.so">
+      <alwaysOn>true</alwaysOn>
+      <bodyName>imu_link</bodyName>
+      <topicName>imu</topicName>
+      <serviceName>imu_service</serviceName>
+      <gaussianNoise>0.0</gaussianNoise>
+      <updateRate>20.0</updateRate>
+    </plugin>
+  </gazebo>
   <!--BASE_LINK-->
   <link
@@ -38,35 +53,35 @@
     <inertial>
       <origin
-        xyz="-0.000103296813793522 -0.0184749995894324 -0.00709986514009202"
-        rpy="0 0 0" />
-      <mass
-        value="0.933836944447792" />
-      <inertia
-        ixx="0.00139201398308306"
-        ixy="-2.82901658884336E-12"
-        ixz="4.14929438991966E-12"
-        iyy="0.00736197315629375"
-        iyz="-8.0885885721078E-10"
-        izz="0.00614175111526735" />
-    </inertial>
-    <visual>
-      <origin
-        xyz="0 0 0"
-        rpy="0 0 0" />
-      <geometry>
-        <mesh
-          filename="package://hmr/hmr_description/meshesbase_link.STL" />
-      </geometry>
-      <material name="red">
-        <color rgba="1.0 0.0 0.0 1.0"/>
-      </material>
-    </visual>
-    <collision>
-      <origin
-        xyz="0 0 0"
-        rpy="0 0 0" />
-      <geometry>
-        <mesh
-          filename="package://hmr/hmr_description/meshesbase_link.STL" />
+        xyz="-8.1485E-05 0.040306 -0.00093209"
+        rpy="0 0 0" />
+      <mass
+        value="2.4018" />
+      <inertia
+        ixx="0.0070769"
+        ixy="-2.7325E-07"
+        ixz="1.9337E-07"
+        iyy="0.015485"
+        iyz="-1.2071E-07"
+        izz="0.009591" />
+    </inertial>
+    <visual>
+      <origin
+        xyz="0 0 0"
+        rpy="0 0 0" />
+      <geometry>
+        <mesh
+          filename="package://hmr/hmr_description/meshes/base_link.STL" />
+      </geometry>
+      <material name="white">
+        <color rgba="1.0 1.0 1.0 1.0"/>
+      </material>
+    </visual>
+    <collision>
+      <origin
+        xyz="0 0 0"
+        rpy="0 0 0" />
+      <geometry>
+        <mesh
+          filename="package://hmr/hmr_description/meshes/base_link.STL" />
       </geometry>
     </collision>
@@ -78,5 +93,6 @@
     <parent link="base"/>
     <child link="base_link"/>
-    <origin xyz="0.0 0.0 1.12" rpy="0.0 0.0 0.0"/>
+    <origin xyz="0.0 0.0 1.4 " rpy="0.0 0.0 3.1416"/>
+    <!-- 1.12 -->
   </joint>
   <!--LLINK1-->
@@ -85,23 +101,23 @@
     <inertial>
       <origin
-        xyz="0.0499999851262689 -0.248500614775013 5.33671345059814E-05"
-        rpy="0 0 0" />
-      <mass
-        value="0.509664464543895" />
-      <inertia
-        ixx="0.00405279295169879"
-        ixy="-5.17821013423379E-16"
-        ixz="-1.86028405386162E-17"
-        iyy="0.000257140430774596"
-        iyz="2.20410095949559E-06"
-        izz="0.0041884713527824" />
-    </inertial>
-    <visual>
-      <origin
-        xyz="0 0 0"
-        rpy="0 0 0" />
-      <geometry>
-        <mesh
-          filename="package://hmr/hmr_description/meshesllink1.STL" />
+        xyz="0.056084 -0.21548 -1.1057E-06"
+        rpy="0 0 0" />
+      <mass
+        value="0.43137" />
+      <inertia
+        ixx="0.0026126"
+        ixy="-1.5474E-07"
+        ixz="-5.4626E-08"
+        iyy="0.00020436"
+        iyz="-9.8E-06"
+        izz="0.0027266" />
+    </inertial>
+    <visual>
+      <origin
+        xyz="0 0 0"
+        rpy="0 0 0" />
+      <geometry>
+        <mesh
+          filename="package://hmr/hmr_description/meshes/llink1.STL" />
       </geometry>
       <material name="blue">
@@ -115,5 +131,5 @@
       <geometry>
         <mesh
-          filename="package://hmr/hmr_description/meshesllink1.STL" />
+          filename="package://hmr/hmr_description/meshes/llink1.STL" />
       </geometry>
     </collision>
@@ -124,7 +140,7 @@
   <joint
     name="ljoint1"
-    type="continuous">
+    type="revolute">
     <origin
-      xyz="0.12 0.06 -0.06"
+      xyz="0.1135 0.04 -0.06"
       rpy="1.5708 0 0" />
     <parent
@@ -134,5 +150,6 @@
     <axis
       xyz="1 0 0" />
-    <limit lower="-0.6981" upper="1.0472" effort="2.0" velocity="0.2"/>
+    <limit lower="-0.6981" upper="0.5236" effort="2.0" velocity="0.2"/>
+    <!-- <safety_controller soft_lower_limit="" soft_upper_limit="" k_position="" k_velocity=""/> -->
   </joint>
   <!--LLINK2-->
@@ -141,23 +158,23 @@
     <inertial>
       <origin
-        xyz="0.0500545282509017 -0.234393633663144 0.00550026352716933"
-        rpy="0 0 0" />
-      <mass
-        value="0.442265777754145" />
-      <inertia
-        ixx="0.0040117979862963"
-        ixy="-5.09697896497051E-16"
-        ixz="-2.77164071387431E-17"
-        iyy="0.000241596436981563"
-        iyz="-1.10278899850188E-06"
-        izz="0.00416183117175302" />
-    </inertial>
-    <visual>
-      <origin
-        xyz="0 0 0"
-        rpy="0 0 0" />
-      <geometry>
-        <mesh
-          filename="package://hmr/hmr_description/meshesllink2.STL" />
+        xyz="0.054446 -0.17796 -0.0015786"
+        rpy="0 0 0" />
+      <mass
+        value="0.45541" />
+      <inertia
+        ixx="0.002625"
+        ixy="6.5245E-19"
+        ixz="-3.637E-17"
+        iyy="0.00023283"
+        iyz="4.9149E-06"
+        izz="0.0027437" />
+    </inertial>
+    <visual>
+      <origin
+        xyz="0 0 0"
+        rpy="0 0 0" />
+      <geometry>
+        <mesh
+          filename="package://hmr/hmr_description/meshes/llink2.STL" />
       </geometry>
       <material name="green">
@@ -171,5 +188,5 @@
       <geometry>
         <mesh
-          filename="package://hmr/hmr_description/meshesllink2.STL" />
+          filename="package://hmr/hmr_description/meshes/llink2.STL" />
       </geometry>
     </collision>
@@ -180,7 +197,7 @@
   <joint
     name="ljoint2"
-    type="continuous">
+    type="revolute">
     <origin
-      xyz="0 -0.5 0"
+      xyz="0 -0.438 0"
       rpy="0 0 0" />
     <parent
@@ -190,5 +207,6 @@
     <axis
       xyz="1 0 0" />
-    <limit lower="-1.0472" upper="0.0" effort="2.0" velocity="0.2"/>
+    <limit lower="0.0" upper="1.0472" effort="2.0" velocity="0.2"/>
+    <!-- <safety_controller soft_lower_limit="" soft_upper_limit="" k_position="" k_velocity=""/> -->
   </joint>
   <!--LLINK3-->
@@ -197,35 +215,35 @@
     <inertial>
       <origin
-        xyz="0.0501466994062446 -0.0351041894822217 0.0405185729509365"
-        rpy="0 0 0" />
-      <mass
-        value="0.164387087553345" />
-      <inertia
-        ixx="0.000390399624612182"
-        ixy="6.46553823154572E-18"
-        ixz="7.16521493881578E-17"
-        iyy="0.000442516689346383"
-        iyz="-8.18654011913839E-11"
-        izz="8.27552994226968E-05" />
-    </inertial>
-    <visual>
-      <origin
-        xyz="0 0 0"
-        rpy="0 0 0" />
-      <geometry>
-        <mesh
-          filename="package://hmr/hmr_description/meshesllink3.STL" />
-      </geometry>
-      <material name="black">
-        <color rgba="0.0 0.0 0.0 1.0"/>
-      </material>
-    </visual>
-    <collision>
-      <origin
-        xyz="0 0 0"
-        rpy="0 0 0" />
-      <geometry>
-        <mesh
-          filename="package://hmr/hmr_description/meshesllink3.STL" />
+        xyz="0.049198 -0.036675 0.049331"
+        rpy="0 0 0" />
+      <mass
+        value="0.29119" />
+      <inertia
+        ixx="0.00061049"
+        ixy="1.3662E-07"
+        ixz="-9.6685E-08"
+        iyy="0.00068435"
+        iyz="-6.0356E-08"
+        izz="0.00011606" />
+    </inertial>
+    <visual>
+      <origin
+        xyz="0 0 0"
+        rpy="0 0 0" />
+      <geometry>
+        <mesh
+          filename="package://hmr/hmr_description/meshes/llink3.STL" />
+      </geometry>
+      <material name="red">
+        <color rgba="1.0 0.0 0.0 1.0"/>
+      </material>
+    </visual>
+    <collision>
+      <origin
+        xyz="0 0 0"
+        rpy="0 0 0" />
+      <geometry>
+        <mesh
+          filename="package://hmr/hmr_description/meshes/llink3.STL" />
       </geometry>
     </collision>
@@ -236,7 +254,7 @@
   <joint
     name="ljoint3"
-    type="continuous">
+    type="revolute">
     <origin
-      xyz="0 -0.5 0"
+      xyz="0.00735 -0.44 0"
       rpy="0 0 0" />
     <parent
@@ -246,5 +264,6 @@
     <axis
       xyz="1 0 0" />
-    <limit lower="-0.8727" upper="0.5236" effort="2.0" velocity="0.2"/>
+    <limit lower="-0.3491" upper="0.8727" effort="2.0" velocity="0.2"/>
+    <!-- <safety_controller soft_lower_limit="" soft_upper_limit="" k_position="" k_velocity=""/> -->
   </joint>
   <!--RLINK1-->
@@ -253,23 +272,23 @@
     <inertial>
       <origin
-        xyz="-0.0500000148736693 -0.248500614774999 5.33671345059189E-05"
-        rpy="0 0 0" />
-      <mass
-        value="0.509664464543895" />
-      <inertia
-        ixx="0.00405279295169879"
-        ixy="-5.17781100332924E-16"
-        ixz="-1.86069004433025E-17"
-        iyy="0.000257140430774596"
-        iyz="2.20410095949557E-06"
-        izz="0.0041884713527824" />
-    </inertial>
-    <visual>
-      <origin
-        xyz="0 0 0"
-        rpy="0 0 0" />
-      <geometry>
-        <mesh
-          filename="package://hmr/hmr_description/meshesrlink1.STL" />
+        xyz="-0.046266 -0.21548 -1.1057E-06"
+        rpy="0 0 0" />
+      <mass
+        value="0.43137" />
+      <inertia
+        ixx="0.0026126"
+        ixy="-1.5474E-07"
+        ixz="-5.4626E-08"
+        iyy="0.00020436"
+        iyz="-9.8E-06"
+        izz="0.0027266" />
+    </inertial>
+    <visual>
+      <origin
+        xyz="0 0 0"
+        rpy="0 0 0" />
+      <geometry>
+        <mesh
+          filename="package://hmr/hmr_description/meshes/rlink1.STL" />
       </geometry>
       <material name="blue">
@@ -283,5 +302,5 @@
       <geometry>
         <mesh
-          filename="package://hmr/hmr_description/meshesrlink1.STL" />
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
Commit message: up

File: hmr_description/urdf/test2.xacro (robot description, xacro)
@@ -14,9 +14,9 @@
     </plugin>
   </gazebo>
-  <link name="world"/>
+  <!-- <link name="world"/>
   <joint name="fixed" type="fixed">
     <parent link="world"/>
     <child link="base"/>
-  </joint>
+  </joint> -->
   <link name="base">
   </link>
@@ -33,4 +33,24 @@
   <link name="imu_link"/>
   <gazebo reference="imu_link">
+    <gravity>true</gravity>
+    <sensor name="imu_sensor" type="imu">
+      <always_on>true</always_on>
+      <update_rate>100</update_rate>
+      <visualize>true</visualize>
+      <topic>__default_topic__</topic>
+      <plugin filename="libgazebo_ros_imu_sensor.so" name="imu_plugin">
+        <topicName>imu/data</topicName>
+        <bodyName>base</bodyName>
+        <updateRateHZ>10.0</updateRateHZ>
+        <gaussianNoise>0.0</gaussianNoise>
+        <xyzOffset>0 0 0</xyzOffset>
+        <rpyOffset>0 0 0</rpyOffset>
+        <frameName>imu_link</frameName>
+        <initialOrientationAsReference>false</initialOrientationAsReference>
+      </plugin>
+      <pose>0 0 0 0 0 0</pose>
+    </sensor>
+  </gazebo>
+  <!-- <gazebo reference="imu_link">
     <sensor type="imu" name="imu">
       <always_on>true</always_on>
@@ -47,5 +67,5 @@
       <updateRate>20.0</updateRate>
     </plugin>
-  </gazebo>
+  </gazebo> -->
   <!--BASE_LINK-->
   <link
@@ -93,5 +113,5 @@
     <parent link="base"/>
     <child link="base_link"/>
-    <origin xyz="0.0 0.0 1.4 " rpy="0.0 0.0 3.1416"/>
+    <origin xyz="0.0 0.0 1.25 " rpy="0.0 0.0 3.1416"/>
     <!-- 1.12 -->
   </joint>

Commit message: up

File: hmr_description/urdf/test2.xacro (robot description, xacro)
@@ -14,9 +14,9 @@
     </plugin>
   </gazebo>
-  <!-- <link name="world"/>
+  <link name="world"/>
   <joint name="fixed" type="fixed">
     <parent link="world"/>
     <child link="base"/>
-  </joint> -->
+  </joint>
   <link name="base">
   </link>

Commit message: up

File: hmr_description/urdf/test2.xacro (robot description, xacro)
@@ -52,20 +52,4 @@
     </sensor>
   </gazebo>
-  <!-- <gazebo reference="imu_link">
-    <sensor type="imu" name="imu">
-      <always_on>true</always_on>
-    </sensor>
-    <material>Gazebo/FlatBlack</material>
-  </gazebo>
-  <gazebo>
-    <plugin name="imu_plugin" filename="libgazebo_ros_imu.so">
-      <alwaysOn>true</alwaysOn>
-      <bodyName>imu_link</bodyName>
-      <topicName>imu</topicName>
-      <serviceName>imu_service</serviceName>
-      <gaussianNoise>0.0</gaussianNoise>
-      <updateRate>20.0</updateRate>
-    </plugin>
-  </gazebo> -->
   <!--BASE_LINK-->
   <link

Commit message: up

File: hmr_description/urdf/test2.xacro (robot description, xacro)
@@ -14,9 +14,9 @@
     </plugin>
   </gazebo>
-  <link name="world"/>
+  <!-- <link name="world"/>
   <joint name="fixed" type="fixed">
     <parent link="world"/>
     <child link="base"/>
-  </joint>
+  </joint> -->
   <link name="base">
   </link>
@@ -27,5 +27,5 @@
     <parent link="base"/>
     <child link="imu_link"/>
-    <origin xyz="0.0 0.0 1.4 " rpy="0.0 0.0 3.1416"/>
+    <origin xyz="0.0 0.0 1.003 " rpy="0.0 0.0 3.1416"/>
     <!-- 1.12 -->
   </joint>
@@ -97,5 +97,5 @@
     <parent link="base"/>
     <child link="base_link"/>
-    <origin xyz="0.0 0.0 1.25 " rpy="0.0 0.0 3.1416"/>
+    <origin xyz="0.0 0.0 1.003 " rpy="0.0 0.0 3.1416"/>
     <!-- 1.12 -->
   </joint>
