Commit message: update

File: hmr_description/urdf/test2_IMU.xacro (robot description, xacro)
@@ -24,11 +24,12 @@
     <material>Gazebo/Blue</material>
   </gazebo>
-  <!-- <joint name="imu_joint" type="fixed">
+  <joint name="imu_joint" type="fixed">
     <parent link="base"/>
     <child link="imu_link"/>
     <origin xyz="0.0 0.0 1.003 " rpy="0.0 0.0 3.1416"/>
-  </joint>   -->
+    <!-- 1.12 -->
+  </joint>
   <!--IMU-->
-  <!-- <link name="imu_link"/>
+  <link name="imu_link"/>
   <gazebo reference="imu_link">
     <gravity>true</gravity>
@@ -50,5 +51,5 @@
       <pose>0 0 0 0 0 0</pose>
     </sensor>
-  </gazebo> -->
+  </gazebo>
   <!--BASE_LINK-->
   <link
