Commit message: update new version

File: hmr_description/urdf/test2_gazebo.xacro (robot description, xacro)
@@ -4,14 +4,7 @@
   xmlns:xacro="http://www.ros.org/wiki/xacro">
   <xacro:property name="PI" value="3.1415926535897931"/>
-  <!-- Import Rviz colors -->
-  <!-- <xacro:include filename="$(find hmr)/urdf/materials.xacro" /> -->
+  <!-- Import Gazebo -->
+  <xacro:include filename="$(find hmr)/hmr_description/urdf/gazebo.xacro" />
   <!-- Import all Gazebo-customization elements, including Gazebo colors -->
-  <!-- <xacro:include filename="$(find hmr)/urdf/test2.gazebo" /> -->
-  <gazebo>
-    <plugin name="gazebo_ros_control" filename="libgazebo_ros_control.so">
-      <robotNamespace>/hmr</robotNamespace>
-      <!-- <robotSimType>gazebo_ros_control/DefaultRobotHWSim</robotSimType> -->
-    </plugin>
-  </gazebo>
   <!-- The ft_sensor plugin -->
   <!-- <gazebo>
@@ -29,7 +22,4 @@
   <link name="base">
   </link>
-  <gazebo reference="base">
-    <material>Gazebo/Blue</material>
-  </gazebo>
   <joint name="imu_joint" type="fixed">
     <parent link="base"/>
@@ -40,24 +30,4 @@
   <!--IMU-->
   <link name="imu_link"/>
-  <gazebo reference="imu_link">
-    <gravity>true</gravity>
-    <sensor name="imu_sensor" type="imu">
-      <always_on>true</always_on>
-      <update_rate>100</update_rate>
-      <visualize>true</visualize>
-      <topic>__default_topic__</topic>
-      <plugin filename="libgazebo_ros_imu_sensor.so" name="imu_plugin">
-        <topicName>imu/data</topicName>
-        <bodyName>base</bodyName>
-        <updateRateHZ>10.0</updateRateHZ>
-        <gaussianNoise>0.0</gaussianNoise>
-        <xyzOffset>0 0 0</xyzOffset>
-        <rpyOffset>0 0 0</rpyOffset>
-        <frameName>imu_link</frameName>
-        <initialOrientationAsReference>false</initialOrientationAsReference>
-      </plugin>
-      <pose>0 0 0 0 0 0</pose>
-    </sensor>
-  </gazebo>
   <!--BASE_LINK-->
   <link
@@ -99,7 +69,4 @@
     </collision>
   </link>
-  <gazebo reference="base_link">
-    <material>Gazebo/Blue</material>
-  </gazebo>
   <joint name="joint" type="fixed">
     <parent link="base"/>
@@ -147,7 +114,4 @@
     </collision>
   </link>
-  <gazebo reference="llink1">
-    <material>Gazebo/Blue</material>
-  </gazebo>
   <joint
     name="ljoint1"
@@ -204,7 +168,4 @@
     </collision>
   </link>
-  <gazebo reference="llink2">
-    <material>Gazebo/Blue</material>
-  </gazebo>
   <joint
     name="ljoint2"
@@ -261,7 +222,4 @@
     </collision>
   </link>
-  <gazebo reference="llink3">
-    <material>Gazebo/Blue</material>
-  </gazebo>
   <joint
     name="ljoint3"
@@ -318,7 +276,4 @@
     </collision>
   </link>
-  <gazebo reference="rlink1">
-    <material>Gazebo/Blue</material>
-  </gazebo>
   <joint
     name="rjoint1"
@@ -375,7 +330,4 @@
     </collision>
   </link>
-  <gazebo reference="rlink2">
-    <material>Gazebo/Blue</material>
-  </gazebo>
   <joint
     name="rjoint2"
@@ -432,7 +384,4 @@
     </collision>
   </link>
-  <gazebo reference="rlink3">
-    <material>Gazebo/Blue</material>
-  </gazebo>
   <joint
     name="rjoint3"

Commit message: up

File: hmr_description/urdf/test2_gazebo.xacro (robot description, xacro)
@@ -29,5 +29,6 @@
   </joint>
   <!--IMU-->
-  <link name="imu_link"/>
+  <link name="imu_link">
+  </link>
   <!--BASE_LINK-->
   <link
