Commit message: up

File: hmr_description/urdf/test2.gazebo.xacro (robot description, xacro)
@@ -6,5 +6,6 @@
   <!-- Import Gazebo -->
   <xacro:include filename="$(find hmr)/hmr_description/urdf/gazebo.xacro" />
-  <!-- Import all Gazebo-customization elements, including Gazebo colors -->
+  <!-- Import Transmission -->
+  <xacro:include filename="$(find hmr)/hmr_description/urdf/transmission.xacro" />
   <!-- The ft_sensor plugin -->
   <!-- <gazebo>
@@ -400,64 +401,3 @@
     <!-- <safety_controller soft_lower_limit="" soft_upper_limit="" k_position="" k_velocity=""/> -->
   </joint>
-  <!--  -->
-  <transmission name="ltran1">
-    <type>transmission_interface/SimpleTransmission</type>
-    <joint name="ljoint1">
-      <hardwareInterface>hardware_interface/EffortJointInterface</hardwareInterface>
-    </joint>
-    <actuator name="lmotor1">
-      <mechanicalReduction>1.0</mechanicalReduction>
-      <hardwareInterface>hardware_interface/EffortJointInterface</hardwareInterface>
-    </actuator>
-  </transmission>
-  <transmission name="ltran2">
-    <type>transmission_interface/SimpleTransmission</type>
-    <joint name="ljoint2">
-      <hardwareInterface>hardware_interface/EffortJointInterface</hardwareInterface>
-    </joint>
-    <actuator name="lmotor2">
-      <mechanicalReduction>1.0</mechanicalReduction>
-      <hardwareInterface>hardware_interface/EffortJointInterface</hardwareInterface>
-    </actuator>
-  </transmission>
-  <transmission name="ltran3">
-    <type>transmission_interface/SimpleTransmission</type>
-    <joint name="ljoint3">
-      <hardwareInterface>hardware_interface/EffortJointInterface</hardwareInterface>
-    </joint>
-    <actuator name="lmotor3">
-      <mechanicalReduction>1.0</mechanicalReduction>
-      <hardwareInterface>hardware_interface/EffortJointInterface</hardwareInterface>
-    </actuator>
-  </transmission>
-  <transmission name="rtran1">
-    <type>transmission_interface/SimpleTransmission</type>
-    <joint name="rjoint1">
-      <hardwareInterface>hardware_interface/EffortJointInterface</hardwareInterface>
-    </joint>
-    <actuator name="rmotor1">
-      <mechanicalReduction>1.0</mechanicalReduction>
-      <hardwareInterface>hardware_interface/EffortJointInterface</hardwareInterface>
-    </actuator>
-  </transmission>
-  <transmission name="rtran2">
-    <type>transmission_interface/SimpleTransmission</type>
-    <joint name="rjoint2">
-      <hardwareInterface>hardware_interface/EffortJointInterface</hardwareInterface>
-    </joint>
-    <actuator name="rmotor2">
-      <mechanicalReduction>1.0</mechanicalReduction>
-      <hardwareInterface>hardware_interface/EffortJointInterface</hardwareInterface>
-    </actuator>
-  </transmission>
-  <transmission name="rtran3">
-    <type>transmission_interface/SimpleTransmission</type>
-    <joint name="rjoint3">
-      <hardwareInterface>hardware_interface/EffortJointInterface</hardwareInterface>
-    </joint>
-    <actuator name="rmotor3">
-      <mechanicalReduction>1.0</mechanicalReduction>
-      <hardwareInterface>hardware_interface/EffortJointInterface</hardwareInterface>
-    </actuator>
-  </transmission>
 </robot>

File: hmr_description/urdf/test2.urdf.xacro (robot description, xacro)
@@ -4,12 +4,7 @@
   xmlns:xacro="http://www.ros.org/wiki/xacro">
   <xacro:property name="PI" value="3.1415926535897931"/>
-  <!-- Import Rviz colors -->
-  <!-- <xacro:include filename="$(find hmr)/urdf/materials.xacro" /> -->
-  <!-- Import all Gazebo-customization elements, including Gazebo colors -->
-  <!-- <xacro:include filename="$(find hmr)/urdf/test2.gazebo" /> -->
   <gazebo>
     <plugin name="gazebo_ros_control" filename="libgazebo_ros_control.so">
       <robotNamespace>/hmr</robotNamespace>
-      <!-- <robotSimType>gazebo_ros_control/DefaultRobotHWSim</robotSimType> -->
     </plugin>
   </gazebo>

Commit message: Update test2.gazebo.xacro

File: hmr_description/urdf/test2.gazebo.xacro (robot description, xacro)
@@ -16,9 +16,9 @@
       </plugin>
   </gazebo> -->
-  <!-- <link name="world"/>
+  <link name="world"/>
   <joint name="fixed" type="fixed">
     <parent link="world"/>
     <child link="base"/>
-  </joint> -->
+  </joint>
   <link name="base">
   </link>
@@ -26,5 +26,5 @@
     <parent link="base"/>
     <child link="imu_link"/>
-    <origin xyz="0.0 0.0 1.003 " rpy="0.0 0.0 3.1416"/>
+    <origin xyz="0.0 0.0 1.4 " rpy="0.0 0.0 3.1416"/>
     <!-- 1.12 -->
   </joint>
@@ -74,6 +74,5 @@
     <parent link="base"/>
     <child link="base_link"/>
-    <origin xyz="0.0 0.0 1.003 " rpy="0.0 0.0 3.1416"/>
-    <!-- 1.12 -->
+    <origin xyz="0.0 0.0 1.4 " rpy="0.0 0.0 3.1416"/>
   </joint>
   <!--LLINK1-->

Commit message: code new

File: hmr_description/urdf/test2.gazebo.xacro (robot description, xacro)
@@ -127,4 +127,5 @@
     <axis
       xyz="1 0 0" />
+    <dynamics damping="100" friction="0.0"/>
     <limit lower="-0.6981" upper="0.5236" effort="2.0" velocity="0.2"/>
     <!-- <safety_controller soft_lower_limit="" soft_upper_limit="" k_position="" k_velocity=""/> -->
@@ -181,4 +182,5 @@
     <axis
       xyz="1 0 0" />
+    <dynamics damping="100" friction="0.0"/>
     <limit lower="0.0" upper="1.0472" effort="2.0" velocity="0.2"/>
     <!-- <safety_controller soft_lower_limit="" soft_upper_limit="" k_position="" k_velocity=""/> -->
@@ -235,4 +237,5 @@
     <axis
       xyz="1 0 0" />
+    <dynamics damping="100" friction="0.0"/>
     <limit lower="-0.3491" upper="0.8727" effort="2.0" velocity="0.2"/>
     <!-- <safety_controller soft_lower_limit="" soft_upper_limit="" k_position="" k_velocity=""/> -->
@@ -289,4 +292,5 @@
     <axis
       xyz="1 0 0" />
+    <dynamics damping="100" friction="0.0"/>
     <limit lower="-0.6981" upper="0.5236" effort="2.0" velocity="0.2"/>
     <!-- <safety_controller soft_lower_limit="" soft_upper_limit="" k_position="" k_velocity=""/> -->
@@ -343,4 +347,5 @@
     <axis
       xyz="1 0 0" />
+    <dynamics damping="100" friction="0.0"/>
     <limit lower="0.0" upper="1.0472" effort="2.0" velocity="0.2"/>
     <!-- <safety_controller soft_lower_limit="" soft_upper_limit="" k_position="" k_velocity=""/> -->
@@ -397,4 +402,5 @@
     <axis
       xyz="1 0 0" />
+    <dynamics damping="100" friction="0.0"/>
     <limit lower="-0.3491" upper="0.8727" effort="2.0" velocity="0.2"/>
     <!-- <safety_controller soft_lower_limit="" soft_upper_limit="" k_position="" k_velocity=""/> -->

File: hmr_description/urdf/test2_inertial.xacro (robot description, xacro)
@@ -119,5 +119,6 @@
     <axis
       xyz="1 0 0" />
-    <limit lower="-0.6981" upper="0.5236" effort="2.0" velocity="0.34906"/>
+    <dynamics damping="10" friction="0.0"/>
+    <limit lower="-0.87266" upper="0.69813" effort="2.0" velocity="1"/>
     <!-- <safety_controller soft_lower_limit="" soft_upper_limit="" k_position="" k_velocity=""/> -->
   </joint>
@@ -173,5 +174,6 @@
     <axis
       xyz="1 0 0" />
-    <limit lower="0.0" upper="1.0472" effort="2.0" velocity="0.34906"/>
+    <dynamics damping="10" friction="0.0"/>
+    <limit lower="0.0" upper="1.13446" effort="2.0" velocity="1"/>
     <!-- <safety_controller soft_lower_limit="" soft_upper_limit="" k_position="" k_velocity=""/> -->
   </joint>
@@ -227,5 +229,6 @@
     <axis
       xyz="1 0 0" />
-    <limit lower="-0.3491" upper="0.8727" effort="2.0" velocity="0.34906"/>
+    <dynamics damping="10" friction="0.0"/>
+    <limit lower="-0.34907" upper="0.69813" effort="2.0" velocity="1"/>
     <!-- <safety_controller soft_lower_limit="" soft_upper_limit="" k_position="" k_velocity=""/> -->
   </joint>
@@ -281,5 +284,6 @@
     <axis
       xyz="1 0 0" />
-    <limit lower="-0.6981" upper="0.5236" effort="2.0" velocity="0.34906"/>
+    <dynamics damping="10" friction="0.0"/>
+    <limit lower="-0.87266" upper="0.69813" effort="2.0" velocity="1"/>
     <!-- <safety_controller soft_lower_limit="" soft_upper_limit="" k_position="" k_velocity=""/> -->
   </joint>
@@ -335,5 +339,6 @@
     <axis
       xyz="1 0 0" />
-    <limit lower="0.0" upper="1.0472" effort="2.0" velocity="0.34906"/>
+    <dynamics damping="10" friction="0.0"/>
+    <limit lower="0.0" upper="1.13446" effort="2.0" velocity="1"/>
     <!-- <safety_controller soft_lower_limit="" soft_upper_limit="" k_position="" k_velocity=""/> -->
   </joint>
@@ -389,5 +394,6 @@
     <axis
       xyz="1 0 0" />
-    <limit lower="-0.3491" upper="0.8727" effort="2.0" velocity="0.34906"/>
+    <dynamics damping="10" friction="0.0"/>
+    <limit lower="-0.34907" upper="0.69813" effort="2.0" velocity="1"/>
     <!-- <safety_controller soft_lower_limit="" soft_upper_limit="" k_position="" k_velocity=""/> -->
   </joint>
