Commit message: update pi

File: hmr_description/urdf/test2_inertial copy.xacro (robot description, xacro)
@@ -3,5 +3,5 @@
   name="hmr"
   xmlns:xacro="http://www.ros.org/wiki/xacro">
-  <xacro:property name="pi" value="3.141592653589793"/>
+  <xacro:property name="PI" value="3.1415926535897931"/>
   <!-- Import Gazebo -->
   <xacro:include filename="$(find hmr)/hmr_description/urdf/gazebo.xacro" />
@@ -120,5 +120,5 @@
       xyz="1 0 0" />
     <dynamics damping="10" friction="0.0"/>
-    <limit lower="${-pi*50}" upper="${pi*40}" effort="2.0" velocity="1"/>
+    <limit lower="-0.87266" upper="0.69813" effort="2.0" velocity="1"/>
     <!-- <safety_controller soft_lower_limit="" soft_upper_limit="" k_position="" k_velocity=""/> -->
   </joint>
@@ -175,5 +175,5 @@
       xyz="1 0 0" />
     <dynamics damping="10" friction="0.0"/>
-    <limit lower="0.0" upper="${pi*65}" effort="2.0" velocity="1"/>
+    <limit lower="0.0" upper="1.13446" effort="2.0" velocity="1"/>
     <!-- <safety_controller soft_lower_limit="" soft_upper_limit="" k_position="" k_velocity=""/> -->
   </joint>
@@ -230,5 +230,5 @@
       xyz="1 0 0" />
     <dynamics damping="10" friction="0.0"/>
-    <limit lower="${-pi*20}" upper="${pi*40}" effort="2.0" velocity="1"/>
+    <limit lower="-0.34907" upper="0.69813" effort="2.0" velocity="1"/>
     <!-- <safety_controller soft_lower_limit="" soft_upper_limit="" k_position="" k_velocity=""/> -->
   </joint>
@@ -285,5 +285,5 @@
       xyz="1 0 0" />
     <dynamics damping="10" friction="0.0"/>
-    <limit lower="${-pi*50}" upper="${pi*40}" effort="2.0" velocity="1"/>
+    <limit lower="-0.87266" upper="0.69813" effort="2.0" velocity="1"/>
     <!-- <safety_controller soft_lower_limit="" soft_upper_limit="" k_position="" k_velocity=""/> -->
   </joint>
@@ -340,5 +340,5 @@
       xyz="1 0 0" />
     <dynamics damping="10" friction="0.0"/>
-    <limit lower="0.0" upper="${pi*65}" effort="2.0" velocity="1"/>
+    <limit lower="0.0" upper="1.13446" effort="2.0" velocity="1"/>
     <!-- <safety_controller soft_lower_limit="" soft_upper_limit="" k_position="" k_velocity=""/> -->
   </joint>
@@ -395,5 +395,5 @@
       xyz="1 0 0" />
     <dynamics damping="10" friction="0.0"/>
-    <limit lower="${-pi*20}" upper="${pi*40}" effort="2.0" velocity="1"/>
+    <limit lower="-0.34907" upper="0.69813" effort="2.0" velocity="1"/>
     <!-- <safety_controller soft_lower_limit="" soft_upper_limit="" k_position="" k_velocity=""/> -->
   </joint>
