Commit message: up

File: hmr_description/urdf/gazebo.xacro (robot description, xacro)
@@ -22,5 +22,4 @@
   </gazebo>
   <!--IMU-->
-  <link name="imu_link"/>
   <gazebo reference="imu_link">
     <gravity>true</gravity>

Commit message: Update gazebo.xacro

File: hmr_description/urdf/gazebo.xacro (robot description, xacro)
@@ -9,15 +9,4 @@
       <!-- <robotSimType>gazebo_ros_control/DefaultRobotHWSim</robotSimType> -->
     </plugin>
-  </gazebo>
-  <!-- The ft_sensor plugin -->
-  <!-- <gazebo>
-      <plugin name="ft_sensor" filename="libgazebo_ros_ft_sensor.so">
-          <updateRate>100.0</updateRate>
-          <topicName>ft_sensor_topic</topicName>
-          <jointName>schunk_wsg50_fixed_base_joint</jointName>
-      </plugin>
-  </gazebo> -->
-  <gazebo reference="base">
-    <material>Gazebo/Blue</material>
   </gazebo>
   <!--IMU-->
@@ -42,4 +31,8 @@
     </sensor>
   </gazebo>
+  <!--BASE-->
+  <gazebo reference="base">
+    <material>Gazebo/Blue</material>
+  </gazebo>
   <!--BASE_LINK-->
   <gazebo reference="base_link">
@@ -50,4 +43,5 @@
     <material>Gazebo/Blue</material>
   </gazebo>
+  <!--F/T-->
   <gazebo reference="ljoint1">
     <provideFeedback>true</provideFeedback>

Commit message: update
Dung vung

File: hmr_description/urdf/gazebo.xacro (robot description, xacro)
@@ -34,12 +34,18 @@
   <gazebo reference="base">
     <material>Gazebo/Blue</material>
+    <mu1>0.2</mu1>
+    <mu2>0.2</mu2>
   </gazebo>
   <!--BASE_LINK-->
   <gazebo reference="base_link">
     <material>Gazebo/Blue</material>
+    <mu1>0.2</mu1>
+    <mu2>0.2</mu2>
   </gazebo>
   <!--LLINK1-->
   <gazebo reference="llink1">
     <material>Gazebo/Blue</material>
+    <mu1>0.2</mu1>
+    <mu2>0.2</mu2>
   </gazebo>
   <!--F/T-->
@@ -57,4 +63,6 @@
   <gazebo reference="llink2">
     <material>Gazebo/Blue</material>
+    <mu1>0.2</mu1>
+    <mu2>0.2</mu2>
   </gazebo>
   <!--F/T-->
@@ -72,4 +80,8 @@
   <gazebo reference="llink3">
     <material>Gazebo/Blue</material>
+    <kp>100000.0</kp>
+    <kd>100.0</kd>
+    <mu1>0.9</mu1>
+    <mu2>0.9</mu2>
   </gazebo>
   <!--F/T-->
@@ -87,4 +99,6 @@
   <gazebo reference="rlink1">
     <material>Gazebo/Blue</material>
+    <mu1>0.2</mu1>
+    <mu2>0.2</mu2>
   </gazebo>
   <!--F/T-->
@@ -102,4 +116,6 @@
   <gazebo reference="rlink2">
     <material>Gazebo/Blue</material>
+    <mu1>0.2</mu1>
+    <mu2>0.2</mu2>
   </gazebo>
   <!--F/T-->
@@ -117,4 +133,8 @@
   <gazebo reference="rlink3">
     <material>Gazebo/Blue</material>
+    <kp>100000.0</kp>
+    <kd>100.0</kd>
+    <mu1>0.9</mu1>
+    <mu2>0.9</mu2>
   </gazebo>
   <!--F/T-->

File: hmr_description/urdf/test2_inertial.xacro (robot description, xacro)
@@ -8,9 +8,9 @@
   <!-- Import Transmission -->
   <xacro:include filename="$(find hmr)/hmr_description/urdf/transmission.xacro" />
-  <link name="world"/>
+  <!-- <link name="world"/>
   <joint name="fixed" type="fixed">
     <parent link="world"/>
     <child link="base"/>
-  </joint>
+  </joint> -->
   <link name="base">
   </link>

Commit message: test ok

File: hmr_description/urdf/gazebo.xacro (robot description, xacro)
@@ -3,5 +3,5 @@
   name="hmr"
   xmlns:xacro="http://www.ros.org/wiki/xacro">
-  <xacro:property name="PI" value="3.1415926535897931"/>
+  <!-- <xacro:property name="PI" value="3.1415926535897931"/> -->
   <gazebo>
     <plugin name="gazebo_ros_control" filename="libgazebo_ros_control.so">

File: hmr_description/urdf/test2_inertial.xacro (robot description, xacro)
@@ -8,9 +8,9 @@
   <!-- Import Transmission -->
   <xacro:include filename="$(find hmr)/hmr_description/urdf/transmission.xacro" />
-  <!-- <link name="world"/>
+  <link name="world"/>
   <joint name="fixed" type="fixed">
     <parent link="world"/>
     <child link="base"/>
-  </joint> -->
+  </joint>
   <link name="base">
   </link>
