Commit message: update

File: hmr_description/urdf/test2_inertial.xacro (robot description, xacro)
@@ -119,5 +119,5 @@
     <axis
       xyz="1 0 0" />
-    <limit lower="-0.6981" upper="0.5236" effort="2.0" velocity="0.2"/>
+    <limit lower="-0.6981" upper="0.5236" effort="2.0" velocity="0.34906"/>
     <!-- <safety_controller soft_lower_limit="" soft_upper_limit="" k_position="" k_velocity=""/> -->
   </joint>
@@ -173,5 +173,5 @@
     <axis
       xyz="1 0 0" />
-    <limit lower="0.0" upper="1.0472" effort="2.0" velocity="0.2"/>
+    <limit lower="0.0" upper="1.0472" effort="2.0" velocity="0.34906"/>
     <!-- <safety_controller soft_lower_limit="" soft_upper_limit="" k_position="" k_velocity=""/> -->
   </joint>
@@ -227,5 +227,5 @@
     <axis
       xyz="1 0 0" />
-    <limit lower="-0.3491" upper="0.8727" effort="2.0" velocity="0.2"/>
+    <limit lower="-0.3491" upper="0.8727" effort="2.0" velocity="0.34906"/>
     <!-- <safety_controller soft_lower_limit="" soft_upper_limit="" k_position="" k_velocity=""/> -->
   </joint>
@@ -281,5 +281,5 @@
     <axis
       xyz="1 0 0" />
-    <limit lower="-0.6981" upper="0.5236" effort="2.0" velocity="0.2"/>
+    <limit lower="-0.6981" upper="0.5236" effort="2.0" velocity="0.34906"/>
     <!-- <safety_controller soft_lower_limit="" soft_upper_limit="" k_position="" k_velocity=""/> -->
   </joint>
@@ -335,5 +335,5 @@
     <axis
       xyz="1 0 0" />
-    <limit lower="0.0" upper="1.0472" effort="2.0" velocity="0.2"/>
+    <limit lower="0.0" upper="1.0472" effort="2.0" velocity="0.34906"/>
     <!-- <safety_controller soft_lower_limit="" soft_upper_limit="" k_position="" k_velocity=""/> -->
   </joint>
@@ -389,5 +389,5 @@
     <axis
       xyz="1 0 0" />
-    <limit lower="-0.3491" upper="0.8727" effort="2.0" velocity="0.2"/>
+    <limit lower="-0.3491" upper="0.8727" effort="2.0" velocity="0.34906"/>
     <!-- <safety_controller soft_lower_limit="" soft_upper_limit="" k_position="" k_velocity=""/> -->
   </joint>

Commit message: UP

File: hmr_description/urdf/test2_inertial.xacro (robot description, xacro)
@@ -120,5 +120,5 @@
       xyz="1 0 0" />
     <dynamics damping="10" friction="0.0"/>
-    <limit lower="${-pi*50}" upper="${pi*40}" effort="2.0" velocity="1"/>
+    <limit lower="${-pi*50}" upper="${pi*40}" effort="1000.0" velocity="3"/>
     <!-- <safety_controller soft_lower_limit="" soft_upper_limit="" k_position="" k_velocity=""/> -->
   </joint>
@@ -175,5 +175,5 @@
       xyz="1 0 0" />
     <dynamics damping="10" friction="0.0"/>
-    <limit lower="0.0" upper="${pi*65}" effort="2.0" velocity="1"/>
+    <limit lower="0.0" upper="${pi*65}" effort="1000.0" velocity="3"/>
     <!-- <safety_controller soft_lower_limit="" soft_upper_limit="" k_position="" k_velocity=""/> -->
   </joint>
@@ -230,5 +230,5 @@
       xyz="1 0 0" />
     <dynamics damping="10" friction="0.0"/>
-    <limit lower="${-pi*20}" upper="${pi*40}" effort="2.0" velocity="1"/>
+    <limit lower="${-pi*20}" upper="${pi*40}" effort="1000.0" velocity="3"/>
     <!-- <safety_controller soft_lower_limit="" soft_upper_limit="" k_position="" k_velocity=""/> -->
   </joint>
@@ -285,5 +285,5 @@
       xyz="1 0 0" />
     <dynamics damping="10" friction="0.0"/>
-    <limit lower="${-pi*50}" upper="${pi*40}" effort="2.0" velocity="1"/>
+    <limit lower="${-pi*50}" upper="${pi*40}" effort="1000.0" velocity="3"/>
     <!-- <safety_controller soft_lower_limit="" soft_upper_limit="" k_position="" k_velocity=""/> -->
   </joint>
@@ -340,5 +340,5 @@
       xyz="1 0 0" />
     <dynamics damping="10" friction="0.0"/>
-    <limit lower="0.0" upper="${pi*65}" effort="2.0" velocity="1"/>
+    <limit lower="0.0" upper="${pi*65}" effort="1000.0" velocity="3"/>
     <!-- <safety_controller soft_lower_limit="" soft_upper_limit="" k_position="" k_velocity=""/> -->
   </joint>
@@ -395,5 +395,5 @@
       xyz="1 0 0" />
     <dynamics damping="10" friction="0.0"/>
-    <limit lower="${-pi*20}" upper="${pi*40}" effort="2.0" velocity="1"/>
+    <limit lower="${-pi*20}" upper="${pi*40}" effort="1000.0" velocity="3"/>
     <!-- <safety_controller soft_lower_limit="" soft_upper_limit="" k_position="" k_velocity=""/> -->
   </joint>

Commit message: update

File: hmr_description/urdf/test2_inertial.xacro (robot description, xacro)
@@ -120,5 +120,5 @@
       xyz="1 0 0" />
     <dynamics damping="10" friction="0.0"/>
-    <limit lower="${-pi*50}" upper="${pi*40}" effort="1000.0" velocity="3"/>
+    <limit lower="${-pi*50}" upper="${pi*40}" effort="1000.0" velocity="2"/>
     <!-- <safety_controller soft_lower_limit="" soft_upper_limit="" k_position="" k_velocity=""/> -->
   </joint>
@@ -175,5 +175,5 @@
       xyz="1 0 0" />
     <dynamics damping="10" friction="0.0"/>
-    <limit lower="0.0" upper="${pi*65}" effort="1000.0" velocity="3"/>
+    <limit lower="0.0" upper="${pi*65}" effort="1000.0" velocity="2"/>
     <!-- <safety_controller soft_lower_limit="" soft_upper_limit="" k_position="" k_velocity=""/> -->
   </joint>
@@ -230,5 +230,5 @@
       xyz="1 0 0" />
     <dynamics damping="10" friction="0.0"/>
-    <limit lower="${-pi*20}" upper="${pi*40}" effort="1000.0" velocity="3"/>
+    <limit lower="${-pi*30}" upper="${pi*40}" effort="1000.0" velocity="2"/>
     <!-- <safety_controller soft_lower_limit="" soft_upper_limit="" k_position="" k_velocity=""/> -->
   </joint>
@@ -285,5 +285,5 @@
       xyz="1 0 0" />
     <dynamics damping="10" friction="0.0"/>
-    <limit lower="${-pi*50}" upper="${pi*40}" effort="1000.0" velocity="3"/>
+    <limit lower="${-pi*50}" upper="${pi*40}" effort="1000.0" velocity="2"/>
     <!-- <safety_controller soft_lower_limit="" soft_upper_limit="" k_position="" k_velocity=""/> -->
   </joint>
@@ -340,5 +340,5 @@
       xyz="1 0 0" />
     <dynamics damping="10" friction="0.0"/>
-    <limit lower="0.0" upper="${pi*65}" effort="1000.0" velocity="3"/>
+    <limit lower="0.0" upper="${pi*65}" effort="1000.0" velocity="2"/>
     <!-- <safety_controller soft_lower_limit="" soft_upper_limit="" k_position="" k_velocity=""/> -->
   </joint>
@@ -395,5 +395,5 @@
       xyz="1 0 0" />
     <dynamics damping="10" friction="0.0"/>
-    <limit lower="${-pi*20}" upper="${pi*40}" effort="1000.0" velocity="3"/>
+    <limit lower="${-pi*30}" upper="${pi*40}" effort="1000.0" velocity="2"/>
     <!-- <safety_controller soft_lower_limit="" soft_upper_limit="" k_position="" k_velocity=""/> -->
   </joint>
